File: board/ioAmp200W.kicad_pcb (KiCad board)
At the start: 2 copper layers, 1.4 x 9.2 mm, 33 parts, among them J1 USB4105-GF-A-120, J2 USB4105-GF-A-120, J4 SM03B-SRSS-TB, U1 RP2350_60QFN, U2 TPS26750SRSMR, U3 TPD4S480RUKR, U4 ADAU1761BCPZ-RL, Y1 ABM8-272-T3

Commit message: work
Parts:
- added H1: MountingHole_Pad_MP, MountingHole:MountingHole_2.2mm_M2_ISO7380_Pad_TopBottom, F.Cu at (102.5, 102.5)
- added H2: MountingHole_Pad_MP, MountingHole:MountingHole_2.2mm_M2_ISO7380_Pad_TopBottom, F.Cu at (147.5, 102.5)
- added H3: MountingHole_Pad_MP, MountingHole:MountingHole_2.2mm_M2_ISO7380_Pad_TopBottom, F.Cu at (147.5, 147.5)
- added H4: MountingHole_Pad_MP, MountingHole:MountingHole_2.2mm_M2_ISO7380_Pad_TopBottom, F.Cu at (102.5, 147.5)
- added J3: AudioJack3_Ground, Connector_Audio:Jack_3.5mm_PJ320D_Horizontal, F.Cu at (108.8, 125.0)
- added J5: Conn_01x02_Socket, Connector_AMASS:AMASS_XT30U-F_1x02_P5.0mm_Vertical, F.Cu at (146.0, 111.0)
- added J6: Conn_01x02_Socket, Connector_AMASS:AMASS_XT30U-F_1x02_P5.0mm_Vertical, F.Cu at (146.0, 139.0)
- moved U4 44.9 mm to (125.0, 134.1)
- moved U2 43.8 mm to (116.8, 143.8)
- moved USB_POWER1 38.0 mm to (102.6, 138.0)
- moved C16 33.0 mm to (138.6, 121.1)
- moved C17 33.0 mm to (138.6, 123.0)
- moved C18 33.0 mm to (138.6, 125.0)
- moved C10 33.0 mm to (135.8, 121.1)
- moved C11 33.0 mm to (135.8, 123.0)
- moved C12 33.0 mm to (135.8, 125.0)
- moved C13 33.0 mm to (135.8, 127.0)
- moved C3 33.0 mm to (132.9, 121.1)
- moved C4 33.0 mm to (132.9, 123.0)
- moved C6 33.0 mm to (132.9, 125.0)
- moved C7 33.0 mm to (132.9, 127.0)
- moved J4 28.4 mm to (136.4, 104.0)
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- renumbered J1 to USB_DATA1, J2 to USB_POWER1
Connections:
- USB_POWER1 pad A1_B12: unconnected-(J2-GND-PadA1_B12) -> GND
- USB_POWER1 pad B1_A12: unconnected-(J2-GND__1-PadB1_A12) -> GND
- USB_POWER1 pad SH1: unconnected-(J2-SHELL_GND-PadSH1) -> GND
- USB_POWER1 pad SH2: unconnected-(J2-SHELL_GND__1-PadSH2) -> GND
- USB_POWER1 pad SH3: unconnected-(J2-SHELL_GND__2-PadSH3) -> GND
- USB_POWER1 pad SH4: unconnected-(J2-SHELL_GND__3-PadSH4) -> GND
Other:
- board size 1.4 x 9.2 mm -> 50 x 50 mm

Commit message: work
Parts:
- added G***: LOGO, LOGO, B.Cu at (104.6, 111.8)
- added G***: LOGO, LOGO, B.Cu at (142.2, 113.2)
- added G***: LOGO, LOGO, B.Cu at (129.5, 146.5)
- added G***: LOGO, LOGO, B.Cu at (107.5, 125.0)
- added G***: LOGO, LOGO, B.Cu at (141.8, 125.0)
- added G***: LOGO, LOGO, B.Cu at (112.2, 146.5)
- added G***: LOGO, LOGO, B.Cu at (142.2, 136.6)
- added G***: LOGO, LOGO, B.Cu at (104.6, 138.0)
- added SW1: SW_Push, Button_Switch_SMD:SW_SPST_TS-1088-xR020, F.Cu at (119.2, 121.6)
- added SW2: SW_Push, Button_Switch_SMD:SW_SPST_TS-1088-xR020, F.Cu at (132.4, 107.4)
- moved C13 25.2 mm to (116.8, 110.4), turned to 180 degrees
- moved C6 23.3 mm to (118.8, 106.4), turned to 90 degrees
- moved C12 22.6 mm to (116.8, 112.8), turned to 180 degrees
- moved C7 22.3 mm to (116.8, 111.6), turned to 180 degrees
- moved C18 20.5 mm to (119.6, 117.4), turned to -90 degrees
- moved C17 17.7 mm to (129.0, 108.2)
- moved C8 17.5 mm to (122.0, 106.4), turned to 90 degrees
- moved R1 15.8 mm to (129.0, 110.6)
- moved C16 15.5 mm to (123.6, 117.4), turned to -90 degrees
- moved C10 14.6 mm to (121.6, 117.4), turned to -90 degrees
- moved C4 14.2 mm to (129.0, 109.4), turned to 180 degrees
- moved R5 14.1 mm to (116.9, 105.2), turned to 180 degrees
- moved C11 13.1 mm to (129.0, 111.8)
- moved R7 10.9 mm to (116.8, 115.2)
- moved J4 10.5 mm to (125.9, 103.7), turned to 180 degrees
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- renumbered J6 to L_OUT1, J5 to R_OUT1, J3 to TRS1
Routing:
- added copper zone on B.Cu, net GND
- added copper zone on F.Cu, net GND
- added copper zone on In1.Cu, net GND
- added copper zone on In2.Cu, net GND
- added copper zone on In3.Cu, net GND
- added copper zone on In4.Cu, net GND
Other:
- copper layers 2 -> 6

Commit message: work
Parts:
- H1, H2, H3, H4: value MountingHole_Pad_MP -> MountingHole; footprint MountingHole:MountingHole_2.2mm_M2_ISO7380_Pad_TopBottom -> MountingHole:MountingHole_2.1mm
- moved R5 15.7 mm to (131.3, 111.5), turned to 0 degrees
- moved J4 13.9 mm to (112.0, 103.5)
- moved C15 12.8 mm to (117.3, 110.2), turned to 180 degrees
- moved C13 11.4 mm to (124.8, 102.2), turned to 90 degrees
- moved SW1 9.16 mm to (116.0, 113.0), turned to 0 degrees
- moved C12 7.56 mm to (117.3, 105.2)
- moved R1 6.32 mm to (131.3, 104.7), turned to 180 degrees
- moved R7 6.22 mm to (117.3, 109.0)
- moved R8 6.22 mm to (117.3, 107.8)
- moved U2 5.34 mm to (120.0, 135.7), turned to 0 degrees
- moved C17 5.26 mm to (131.3, 103.5)
- moved C7 5.12 mm to (117.3, 106.5)
- moved C11 5.08 mm to (131.3, 107.2)
- moved L1 4.92 mm to (117.3, 103.5), turned to 180 degrees
- moved C14 4.73 mm to (122.3, 102.2)
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
Commit message: work
Parts:
- moved C11 1.76 mm to (133.0, 107.2)
- moved C17 1.76 mm to (133.0, 103.5)
- moved C4 1.76 mm to (133.0, 106.0)
- moved R1 1.76 mm to (133.0, 104.7)
- moved C3 1.76 mm to (133.0, 110.0)
- moved R2 1.76 mm to (133.0, 108.8)
- moved R5 1.76 mm to (133.0, 111.2)
- moved SW2 1.74 mm to (137.8, 104.5)
- moved Y1 1.74 mm to (136.4, 109.1)
- moved SW1 1.50 mm to (116.0, 114.5)
- moved L1 0.99 mm to (118.2, 103.5), turned to 0 degrees
- moved U1 0.39 mm to (125.0, 108.0)
- moved C12 0.25 mm to (117.3, 105.5)
- moved C15 0.25 mm to (117.3, 110.5)
- moved C7 0.25 mm to (117.3, 106.8)
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Connections:
- U1 pad 40: /GPIO26_ADC0 -> GND
- U1 pad 41: /GPIO27_ADC1 -> GND
- U1 pad 42: /GPIO28_ADC2 -> GND
- U1 pad 43: /GPIO29_ADC3 -> GND
Routing:
- net +3V3: track 0.00 -> 6.37 mm
- net GND: track 0.00 -> 5.13 mm
- net +1V1: track 0.00 -> 2.42 mm

Commit message: work
Parts:
- moved C11 1.75 mm to (132.9, 109.0)
- moved C17 1.75 mm to (132.9, 105.2)
- moved C4 1.75 mm to (132.9, 107.7)
- moved R1 1.75 mm to (132.9, 106.5)
- moved C3 1.75 mm to (132.9, 111.7)
- moved R2 1.75 mm to (132.9, 110.5)
- moved R5 1.75 mm to (132.9, 113.0)
- moved C16 0.93 mm to (126.8, 116.0)
- moved SW2 0.30 mm to (137.7, 104.8)
Routing:
- net /GPIO25: track 0.00 -> 10.7 mm
- net +3V3: track 6.37 -> 12.2 mm
- net /GPIO24: track 0.00 -> 5.78 mm
- net /GPIO23: track 0.00 -> 5.72 mm
- net /GPIO10: track 0.00 -> 5.59 mm
- net /GPIO6: track 0.00 -> 5.05 mm
- net /GPIO7: track 0.00 -> 5.05 mm
- net /GPIO22: track 0.00 -> 4.79 mm
- net /GPIO8: track 0.00 -> 4.29 mm
- net /GPIO21: track 0.00 -> 3.79 mm
- net +1V1: track 2.42 -> 5.77 mm
- net /GPIO9: track 0.00 -> 3.21 mm
- net /GPIO20: track 0.00 -> 3.13 mm
- net /GPIO11: track 0.00 -> 2.74 mm
- net /GPIO5: track 0.00 -> 2.50 mm
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
Commit message: switch_dsp
Parts:
- U4: value ADAU1761BCPZ-RL -> TLV320AIC3204IRHBR; footprint adau1761:CP-32-4_ADI -> TLV320AIC3204IRHBR:QFN50P500X500X100-33N
- moved U4 4.79 mm to (120.3, 124.0)

Commit message: work
Parts:
- U4: value TLV320AIC3204IRHBR -> TLV320AIC3256
Changed lines of the file:
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@@
 			)
 		)
-		(property "Value" "TLV320AIC3204IRHBR"
-			(at 10.23 4.035 0)
+		(property "Value" "TLV320AIC3256"
+			(at 5.435 4.035 0)
 			(layer "F.Fab")
+			(hide yes)
 			(effects
 				(font

Commit message: work
Parts:
- added U5: MA5332MS, Library:IFX-PG-IQFN-42-1-V, F.Cu at (135.8, 124.9)
- moved SW2 0.30 mm to (137.7, 104.5)
Connections:
- U2 pad 1: unconnected-(U2-LDO_3V3-Pad1) -> +3V3
- U4 pad 17: unconnected-(U4-AVSS-Pad17) -> GND
- U4 pad 28: unconnected-(U4-DVSS-Pad28) -> GND
- U4 pad 33: unconnected-(U4-EP-Pad33) -> GND
- U4 pad 7: unconnected-(U4-IOVSS-Pad7) -> GND
