File: board/ioAmp200W.kicad_pcb (KiCad board)
At the start: 6 copper layers, 50 x 50 mm, 51 parts, among them J4 SM03B-SRSS-TB, SW1 SW_Push, SW2 SW_Push, U1 RP2350_60QFN, U2 TPS26750SRSMR, U3 TPD4S480RUKR, U4 TLV320AIC3256, U5 MA5332MS, Y1 ABM8-272-T3

Commit message: work
Parts:
- added J1: HUB75 Connector, Connector_IDC:IDC-Header_2x08_P2.54mm_Vertical_SMD, F.Cu at (6.83, 14.5)
- moved U5 9.85 mm to (133.3, 134.4)

Commit message: work
Parts:
- removed J1: HUB75 Connector, Connector_IDC:IDC-Header_2x08_P2.54mm_Vertical_SMD
- added HUB75: Conn_02x08_Odd_Even, Connector_IDC:IDC-Header_2x08_P2.54mm_Vertical_SMD, B.Cu at (130.1, 125.0)
- moved G*** 28.1 mm to (125.0, 102.5)
- moved U5 3.37 mm to (130.3, 135.9)

Commit message: work
Parts:
- moved Y1 3.00 mm to (136.3, 112.1), turned to -90 degrees
- moved SW2 2.33 mm to (136.5, 106.5), turned to -90 degrees
Changed lines of the file:
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@@
 	(footprint "Button_Switch_SMD:SW_SPST_TS-1088-xR020"
 		(layer "F.Cu")
-		(at 137.7 104.5)
+		(at 136.5 106.5 -90)
 		(descr "SMD Tactile Switch, 3.9x3x2 mm, https://lcsc.com/datasheet/lcsc_datasheet_2504101957_XUNPU-TS-1088-AR02016_C720477.pdf")
 		(tags "Tactile Switch")
 		(property "Reference" "SW2"
-			(at 0 -2.65 0)
+			(at 0 -2.65 90)
 			(layer "F.SilkS")
 			(hide yes)
@@
 		)
 		(property "Value" "SW_Push"
-			(at 0 2.65 0)
+			(at 0 2.65 90)
 			(layer "F.Fab")
 			(hide yes)
@@
 		)
 		(property "Datasheet" "~"
-			(at 0 0 0)
+			(at 0 0 270)
 			(unlocked yes)
 			(layer "F.Fab")
@@
 		)
 		(property "Description" ""
-			(at 0 0 0)
+			(at 0 0 270)
 			(unlocked yes)
 			(layer "F.Fab")
@@
 		(attr smd)
 		(fp_line
-			(start -2.1 -1.65)
-			(end 2.1 -1.65)
+			(start -2.1 1.65)
+			(end 2.1 1.65)
 			(stroke
 				(width 0.12)
@@
 		)
 		(fp_line
-			(start -2.1 -1.26)
-			(end -2.1 -1.65)
+			(start 2.1 1.65)
+			(end 2.1 1.26)
 			(stroke
 				(width 0.12)
@@
 		)
 		(fp_line
-			(start -2.1 1.65)
-			(end 2.1 1.65)
+			(start -2.1 -1.26)
+			(end -2.1 -1.65)
 			(stroke
 				(width 0.12)
@@
 		)
 		(fp_line
-			(start 2.1 -1.65)
-			(end 2.1 -1.26)
+			(start -2.1 -1.65)
+			(end 2.1 -1.65)
 			(stroke
 				(width 0.12)
@@
 		)
 		(fp_line
-			(start 2.1 1.65)
-			(end 2.1 1.26)
+			(start 2.1 -1.65)
+			(end 2.1 -1.26)
 			(stroke
 				(width 0.12)
@@
 		)
 		(fp_line
-			(start -3 -1.75)
-			(end -3 1.75)
+			(start -3 1.75)
+			(end 3 1.75)
 			(stroke
 				(width 0.05)
@@
 		)
 		(fp_line
-			(start -3 1.75)
-			(end 3 1.75)
+			(start 3 1.75)
+			(end 3 -1.75)
 			(stroke
 				(width 0.05)
@@
 		)
 		(fp_line
-			(start 3 -1.75)
-			(end -3 -1.75)
+			(start -3 -1.75)
+			(end -3 1.75)
 			(stroke
 				(width 0.05)
@@
 		)
 		(fp_line
-			(start 3 1.75)
-			(end 3 -1.75)
+			(start 3 -1.75)
+			(end -3 -1.75)
 			(stroke
 				(width 0.05)
@@
 		)
 		(fp_line
-			(start -1.95 -1.5)
-			(end 1.95 -1.5)
+			(start -1.95 1.5)
+			(end 1.95 1.5)
 			(stroke
 				(width 0.1)
@@
 		)
 		(fp_line
-			(start -1.95 1.5)
-			(end 1.95 1.5)
+			(start -1.95 -1.5)
+			(end 1.95 -1.5)
 			(stroke
 				(width 0.1)
@@
 		)
 		(pad "1" smd roundrect
-			(at -2.225 0)
+			(at -2.225 0 270)
 			(size 1.05 2)
 			(layers "F.Cu" "F.Mask" "F.Paste")
@@
 		)
 		(pad "2" smd roundrect
-			(at 2.225 0)
+			(at 2.225 0 270)
 			(size 1.05 2)
 			(layers "F.Cu" "F.Mask" "F.Paste")
@@
 	(footprint "Crystal:Crystal_SMD_3225-4Pin_3.2x2.5mm"
 		(layer "F.Cu")
-		(at 136.4 109.1 90)
+		(at 136.35 112.1 -90)
 		(descr "SMD3225/4, Crystal, 3.2x2.5mm package, SMD, generated with kicad-footprint-generator make_crystal.py, http://www.txccrystal.com/images/pdf/7m-accuracy.pdf")
 		(property "Reference" "Y1"
@@
 		(attr smd)
 		(fp_line
-			(start -2.06 -1.71)
-			(end -2.06 1.71)
+			(start -2.06 1.71)
+			(end 2.06 1.71)
 			(stroke
 				(width 0.12)
@@
 		)
 		(fp_line
-			(start -2.06 1.71)
-			(end 2.06 1.71)
+			(start -2.06 -1.71)
+			(end -2.06 1.71)
 			(stroke
 				(width 0.12)
@@
 		)
 		(pad "1" smd roundrect
-			(at -1.1 0.85 90)
+			(at -1.1 0.85 270)
 			(size 1.4 1.2)
 			(layers "F.Cu" "F.Mask" "F.Paste")
@@
 		)
 		(pad "2" smd roundrect
-			(at 1.1 0.85 90)
+			(at 1.1 0.85 270)
 			(size 1.4 1.2)
 			(layers "F.Cu" "F.Mask" "F.Paste")
@@
 		)
 		(pad "3" smd roundrect
-			(at 1.1 -0.85 90)
+			(at 1.1 -0.85 270)
 			(size 1.4 1.2)
 			(layers "F.Cu" "F.Mask" "F.Paste")
@@
 		)
 		(pad "4" smd roundrect
-			(at -1.1 -0.85 90)
+			(at -1.1 -0.85 270)
 			(size 1.4 1.2)
 			(layers "F.Cu" "F.Mask" "F.Paste")
@@
 		(tags "SMD vertical IDC box header  2x08 2.54mm double row")
 		(property "Reference" "HUB75"
-			(at 0 14.97 90)
+			(at 0 14.97 270)
 			(layer "B.SilkS")
 			(hide yes)
@@
 		)
 		(property "Value" "Conn_02x08_Odd_Even"
-			(at 0 -14.97 90)
+			(at 0 -14.97 270)
 			(layer "B.Fab")
 			(hide yes)
@@
 		)
 		(property "Datasheet" "~"
-			(at 0 0 90)
+			(at 0 0 270)
 			(layer "B.Fab")
 			(hide yes)
@@
 		)
 		(property "Description" "Generic connector, double row, 02x08, odd/even pin numbering scheme (row 1 odd numbers, row 2 even numbers), script generated (kicad-library-utils/schlib/autogen/connector/)"
-			(at 0 0 90)
+			(at 0 0 270)
 			(layer "B.Fab")
 			(hide yes)
@@
 		(sheetname "/")
 		(sheetfile "ioAmp200W.kicad_sch")
-		(attr smd)
+		(attr smd exclude_from_bom dnp)
 		(fp_line
 			(start 4.585 -14.08)
 			(end 4.585 -9.9)
 			(stroke
-				(width 0.12)
+				(width 0.25)
 				(type solid)
 			)
@@
 			(end 4.585 -14.08)
 			(stroke
-				(width 0.12)
+				(width 0.25)
 				(type solid)
 			)
@@
 			(end -4.585 -14.08)
 			(stroke
-				(width 0.12)
+				(width 0.25)
+				(type solid)
+			)
+			(layer "B.SilkS")
+		)
+		(fp_line
+			(start -7 1.5)
+			(end -7 -1.5)
+			(stroke
+				(width 0.25)
 				(type solid)
 			)
@@
 			(end -6.085 9.9)
 			(stroke
-				(width 0.12)
+				(width 0.25)
 				(type solid)
 			)
@@
 			(end -4.585 14.08)
 			(stroke
-				(width 0.12)
+				(width 0.25)
 				(type solid)
 			)
@@
 			(end 4.585 9.9)
 			(stroke
-				(width 0.12)
+				(width 0.25)
 				(type solid)
 			)
@@
 			(end 4.585 14.08)
 			(stroke
-				(width 0.12)
+				(width 0.25)
 				(type solid)
 			)

Commit message: work
Parts:
- moved U5 11.9 mm to (135.0, 125.0)
- moved USB_DATA1 0.40 mm to (103.0, 112.0)
- moved USB_POWER1 0.40 mm to (103.0, 138.0)
- moved R3 0.25 mm to (110.2, 113.8)
- moved R4 0.25 mm to (110.2, 110.8)
Connections:
- R3 pad 1: unconnected-(R3-Pad1) -> GND
- R4 pad 1: unconnected-(R4-Pad1) -> GND

Commit message: lib
Parts:
- removed USB_DATA1, USB_POWER1: USB4105-GF-A-120, USB4105_GF_A_120:GCT_USB4105-GF-A-120
- added J1: USB4105-GF-A-120, USB4105_GF_A_120:GCT_USB4105-GF-A-120, F.Cu at (102.8, 112.0)
- added J2: USB4105-GF-A-120, USB4105_GF_A_120:GCT_USB4105-GF-A-120, F.Cu at (102.8, 138.0)
- U2: footprint TI2:VQFN32_RSM_TEX -> TPS26750SRSMR:VQFN32_RSM_TEX-L
- U3: footprint TI:RUK0020B-MFG -> TPD4S480RUKR:RUK0020B-MFG
- U4: value TLV320AIC3256 -> TLV320AIC3254IRHBT; footprint TLV320AIC3204IRHBR:QFN50P500X500X100-33N -> TLV320AIC3254IRHBT:IC_ADS125H01IRHBT
- U5: footprint Library:IFX-PG-IQFN-42-1-V -> MA5332MS_footprint:IFX-PG-IQFN-42-1-V
- moved U4 0.92 mm to (120.5, 124.9)
- moved U5 0.88 mm to (135.8, 124.6)
- moved U2 0.54 mm to (120.3, 136.2)
- moved U3 0.10 mm to (114.8, 141.3)
Connections:
- U4 pad 33: GND -> unconnected-(U4-EP-Pad33)

Commit message: level_shift
Parts:
- removed R1: 1k, Resistor_SMD:R_0402_1005Metric
- removed SW2: SW_Push, Button_Switch_SMD:SW_SPST_TS-1088-xR020
- added C1: 100n, Capacitor_SMD:C_0402_1005Metric, F.Cu at (128.2, 117.5)
- added C19: 100n, Capacitor_SMD:C_0402_1005Metric, F.Cu at (132.0, 111.5)
- added C20: 100n, Capacitor_SMD:C_0402_1005Metric, F.Cu at (118.8, 110.8)
- added C5: 100n, Capacitor_SMD:C_0402_1005Metric, F.Cu at (135.2, 117.6)
- added U6: SN74AHCT245RGYR, Package_DFN_QFN:DHVQFN-20-1EP_2.5x4.5mm_P0.5mm_EP1x3mm, F.Cu at (131.8, 117.6)
- added U7: SN74AHCT245RGYR, Package_DFN_QFN:DHVQFN-20-1EP_2.5x4.5mm_P0.5mm_EP1x3mm, F.Cu at (138.8, 117.6)
- moved R5 16.8 mm to (120.0, 102.2), turned to -90 degrees
- moved C12 14.8 mm to (132.0, 107.2), turned to 0 degrees
- moved U5 8.13 mm to (134.3, 132.6)
- moved Y1 2.81 mm to (135.8, 109.3), turned to 90 degrees
- moved C15 2.75 mm to (120.0, 110.8), turned to -90 degrees
- moved C17 2.46 mm to (130.5, 104.8)
- moved SW1 1.94 mm to (114.8, 116.0)
- moved C9 1.89 mm to (119.0, 102.2), turned to 90 degrees
- moved C3 1.57 mm to (133.5, 110.2), turned to 90 degrees
- moved R2 1.54 mm to (132.0, 109.2)
- moved L1 1.46 mm to (117.5, 104.8), turned to 180 degrees
- moved C11 1.19 mm to (132.0, 108.2)
- moved C4 0.80 mm to (133.5, 108.2), turned to 90 degrees
- moved R8 0.80 mm to (118.0, 107.8)
- moved C7 0.78 mm to (118.0, 106.5)
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Connections:
- U1 pad 26: /RUN -> +3V3
- U3 pad 13: unconnected-(U3-GND-Pad13) -> GND
- U3 pad 18: unconnected-(U3-GND-Pad18) -> GND
- U3 pad 21: unconnected-(U3-Thermal_Pad-Pad21) -> GND
- U3 pad 8: unconnected-(U3-GND-Pad8) -> GND
Routing:
- net +3V3: track 12.2 -> 55.6 mm, vias 0 -> 4
- net GND: track 5.13 -> 27.7 mm, vias 0 -> 7
- net /GPIO16: track 0.00 -> 11.8 mm
- net /GPIO17: track 0.00 -> 11.6 mm
- net /GPIO18: track 0.00 -> 11.5 mm
- net /GPIO23: track 5.72 -> 17.2 mm
- net /GPIO19: track 2.36 -> 13.3 mm
- net /GPIO20: track 3.13 -> 13.9 mm
- net /GPIO21: track 3.79 -> 14.6 mm
- net /GPIO24: track 5.78 -> 16.5 mm
- net /GPIO22: track 4.79 -> 15.4 mm
- net /XIN: track 0.00 -> 9.71 mm
- net +1V1: track 5.77 -> 14.8 mm
- net /VREG_LX: track 0.00 -> 7.44 mm
- net /GPIO25: track 10.7 -> 17.0 mm
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
Commit message: work
Parts:
- moved R4 2.07 mm to (110.0, 108.8), turned to -135 degrees
- moved C5 1.96 mm to (136.2, 115.9)
- moved U7 1.96 mm to (139.8, 115.9)
- moved U6 1.73 mm to (132.5, 116.0)
- moved C1 1.64 mm to (129.0, 116.1)
- moved C16 0.77 mm to (126.5, 115.3)
- moved C2 0.71 mm to (106.8, 105.0), turned to 180 degrees
- moved R3 0.35 mm to (110.0, 113.5)
- moved J4 0.25 mm to (112.0, 103.2)
Routing:
- net /USB_D-: track 0.00 -> 14.7 mm
- net /USB_D+: track 0.00 -> 13.4 mm
- net GND: track 27.7 -> 39.9 mm, vias 7 -> 15
- net /GPIO25: track 17.0 -> 28.0 mm
- net /GPIO24: track 16.5 -> 26.5 mm
- net /GPIO23: track 17.2 -> 26.5 mm
- net /GPIO22: track 15.4 -> 23.9 mm
- net /GPIO21: track 14.6 -> 22.5 mm
- net /GPIO20: track 13.9 -> 21.2 mm
- net /GPIO19: track 13.3 -> 19.9 mm
- net +5V: track 0.00 -> 6.07 mm
- net /GPIO18: track 11.5 -> 17.4 mm
- net /GPIO17: track 11.6 -> 17.0 mm
- net /GPIO16: track 11.8 -> 16.3 mm
- net +3V3: track 55.6 -> 51.7 mm
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
Commit message: work
Parts:
- moved U4 5.51 mm to (119.0, 119.6)
- moved SW1 4.25 mm to (114.8, 111.8)
- moved C18 3.25 mm to (119.2, 114.0), turned to 180 degrees
- moved R6 3.02 mm to (119.2, 112.5), turned to 180 degrees
- moved R5 2.14 mm to (118.0, 101.5), turned to 0 degrees
- moved R3 2.00 mm to (110.0, 111.5), turned to -135 degrees
- moved C9 1.12 mm to (118.0, 102.8), turned to 180 degrees
- moved C8 0.89 mm to (124.2, 101.8)
- moved C14 0.76 mm to (121.5, 102.2)
- moved C13 0.69 mm to (125.2, 101.8)
- moved C6 0.56 mm to (120.5, 102.2)
Routing:
- net /SWD: track 1.02 -> 25.0 mm, vias 1 -> 2
- net /SWCLK: track 1.02 -> 22.2 mm, vias 1 -> 2
- net +3V3: track 51.7 -> 60.9 mm
- net GND: track 39.9 -> 37.1 mm, vias 15 -> 9
- net /QSPI_SS: track 0.00 -> 2.51 mm
- net /~{USB_BOOT}: track 0.00 -> 2.08 mm
- net Net-(J1-CC2): track 2.09 -> 3.26 mm
- net Net-(J1-CC1): track 3.88 -> 3.00 mm
- net /VREG_AVDD: track 4.55 -> 5.36 mm
- net /USB_D-: track 14.7 -> 14.2 mm
