File: board/ioAmp200W.kicad_pcb (KiCad board)
At the start: 6 copper layers, 50 x 50 mm, 59 parts, among them J1 USB4105-GF-A-120, J2 USB4105-GF-A-120, J4 SM03B-SRSS-TB, SW1 SW_Push, U1 RP2350_60QFN, U2 TPS26750SRSMR, U3 TPD4S480RUKR, U4 TLV320AIC3254IRHBT, U5 MA5332MS, U6 SN74AHCT245RGYR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

Commit message: flash
Parts:
- removed R10: 0, Resistor_SMD:R_0402_1005Metric
- removed R9: DNF, Resistor_SMD:R_0402_1005Metric
- R1: value DNF -> 10k
- moved R1 2.85 mm to (112.8, 112.8), turned to -90 degrees
- moved R6 2.80 mm to (112.8, 115.0)
- moved SW1 0.47 mm to (105.0, 119.8)
Connections:
- R1 pad 2: /FLASH_SS -> /QSPI_SS
- U8 pad 1: /FLASH_SS -> /QSPI_SS
Routing:
- net /~{USB_BOOT}: track 0.00 -> 7.26 mm
- net /QSPI_SS: track 8.60 -> 14.5 mm
- net +3V3: track 71.5 -> 75.4 mm
- net /GPIO0: track 4.23 -> 6.48 mm
- net +5V: track 9.04 -> 9.65 mm
- net GND: vias 21 -> 22

Commit message: flash
Connections:
- U1 pad 28: /B1 -> /ROW_E
- U1 pad 29: /ROW_A -> /B1
- U1 pad 31: /ROW_B -> /ROW_A
- U1 pad 32: /ROW_C -> /ROW_B
- U1 pad 33: /ROW_D -> /ROW_C
- U1 pad 34: /ROW_E -> /ROW_D
- U6 pad 11: /ROW_B -> /ROW_A
- U6 pad 12: /ROW_A -> /B1
- U6 pad 13: /B1 -> /ROW_E
- U6 pad 7: /B1_5V -> /ROW_E_5V
- U6 pad 8: /ROW_A_5V -> /B1_5V
- U6 pad 9: /ROW_B_5V -> /ROW_A_5V
- U7 pad 16: /ROW_E -> /ROW_D
- U7 pad 17: /ROW_D -> /ROW_C
- U7 pad 18: /ROW_C -> /ROW_B
- U7 pad 2: /ROW_C_5V -> /ROW_B_5V
- U7 pad 3: /ROW_D_5V -> /ROW_C_5V
- U7 pad 4: /ROW_E_5V -> /ROW_D_5V
Routing:
- net /ROW_E_5V: track 23.0 -> 10.6 mm
- net /ROW_E: track 25.2 -> 20.9 mm
- net /ROW_A: track 21.8 -> 24.7 mm
- net /ROW_B: track 24.7 -> 22.6 mm
- net /ROW_B_5V: track 9.94 -> 11.8 mm
- net /ROW_C: track 22.6 -> 24.0 mm
- net GND: track 65.7 -> 64.3 mm
- net /ROW_D: track 24.0 -> 25.2 mm
- net /ROW_D_5V: track 10.3 -> 11.3 mm
- net /B1: track 20.9 -> 21.8 mm
- net /B1_5V: track 11.3 -> 12.2 mm
- net /SWCLK: track 20.7 -> 21.4 mm

Commit message: hub75
Parts:
- moved L_OUT1 3.00 mm to (146.0, 142.0)
- moved R_OUT1 3.00 mm to (146.0, 108.0)
- moved HUB75 2.89 mm to (133.0, 123.0)
Routing:
- net /R0_5V: track 16.0 -> 12.5 mm
- net /B0_5V: track 14.7 -> 11.3 mm
- net /G0_5V: track 15.9 -> 13.3 mm, vias 1 -> 2
- net /CLK_5V: track 10.6 -> 13.3 mm
- net /OE_5V: track 11.1 -> 13.7 mm
- net /G1_5V: track 12.3 -> 10.2 mm
- net /B1_5V: track 12.2 -> 10.0 mm
- net /R1_5V: track 12.6 -> 10.5 mm
- net /STB_5V: track 10.2 -> 12.0 mm
- net /ROW_C_5V: track 10.7 -> 12.1 mm
- net /ROW_B_5V: track 11.8 -> 10.7 mm
- net /ROW_E_5V: track 10.6 -> 9.95 mm
- net /ROW_A_5V: track 10.3 -> 10.9 mm
- net GND: vias 22 -> 21

Commit message: hub75
Routing:
- net GND: track 64.3 -> 70.8 mm, vias 21 -> 25
- net /G0_5V: vias 2 -> 1

Commit message: work
Parts:
- moved SW1 7.62 mm to (111.5, 115.7), turned to 90 degrees
- moved R6 3.72 mm to (111.5, 111.5)
- moved R1 1.25 mm to (112.8, 111.5)
- moved U4 0.15 mm to (119.2, 122.8)
Routing:
- net /~{USB_BOOT}: track 7.26 -> 1.49 mm
- net /QSPI_SS: track 14.5 -> 17.1 mm
- net +3V3: track 75.4 -> 72.9 mm
- net GND: track 70.8 -> 71.8 mm, vias 25 -> 24
Changed lines of the file:
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@@
 	(footprint "Resistor_SMD:R_0402_1005Metric"
 		(layer "F.Cu")
-		(at 112.75 112.75 -90)
+		(at 112.75 111.5 -90)
 		(descr "Resistor SMD 0402 (1005 Metric), square (rectangular) end terminal, IPC-7351 nominal, (Body size source: IPC-SM-782 page 72, https://www.pcb-3d.com/wordpress/wp-content/uploads/ipc-sm-782a_amendment_1_and_2.pdf), generated with kicad-footprint-generator")
 		(tags "resistor")
@@
 	(footprint "TLV320AIC3254IRHBT:IC_ADS125H01IRHBT"
 		(layer "F.Cu")
-		(at 119.1 122.75 -90)
+		(at 119.25 122.75 -90)
 		(property "Reference" "U4"
 			(at -0.57 -3.723 90)
@@
 	(footprint "Resistor_SMD:R_0402_1005Metric"
 		(layer "F.Cu")
-		(at 112.75 115 -90)
+		(at 111.5 111.5 -90)
 		(descr "Resistor SMD 0402 (1005 Metric), square (rectangular) end terminal, IPC-7351 nominal, (Body size source: IPC-SM-782 page 72, https://www.pcb-3d.com/wordpress/wp-content/uploads/ipc-sm-782a_amendment_1_and_2.pdf), generated with kicad-footprint-generator")
 		(tags "resistor")
@@
 	(footprint "Button_Switch_SMD:SW_SPST_TS-1088-xR020"
 		(layer "F.Cu")
-		(at 105.025 119.75)
+		(at 111.5 115.725 90)
 		(descr "SMD Tactile Switch, 3.9x3x2 mm, https://lcsc.com/datasheet/lcsc_datasheet_2504101957_XUNPU-TS-1088-AR02016_C720477.pdf")
 		(tags "Tactile Switch")
 		(property "Reference" "SW1"
-			(at 0 0 0)
+			(at 0 0 90)
 			(layer "F.SilkS")
 			(hide yes)
@@
 		)
 		(property "Value" "SW_Push"
-			(at 0 2.65 0)
+			(at 0 2.65 90)
 			(layer "F.Fab")
 			(hide yes)
@@
 		)
 		(property "Datasheet" "~"
-			(at 0 0 0)
+			(at 0 0 90)
 			(unlocked yes)
 			(layer "F.Fab")
@@
 		)
 		(property "Description" ""
-			(at 0 0 0)
+			(at 0 0 90)
 			(unlocked yes)
 			(layer "F.Fab")
@@
 		(attr smd)
 		(fp_line
+			(start 2.1 -1.65)
+			(end 2.1 -1.26)
+			(stroke
+				(width 0.12)
+				(type solid)
+			)
+			(layer "F.SilkS")
+		)
+		(fp_line
 			(start -2.1 -1.65)
 			(end 2.1 -1.65)
@@
 		)
 		(fp_line
-			(start -2.1 1.65)
-			(end 2.1 1.65)
+			(start 2.1 1.65)
+			(end 2.1 1.26)
 			(stroke
 				(width 0.12)
@@
 		)
 		(fp_line
-			(start 2.1 -1.65)
-			(end 2.1 -1.26)
+			(start -2.1 1.65)
+			(end 2.1 1.65)
 			(stroke
 				(width 0.12)
@@
 		)
 		(fp_line
-			(start 2.1 1.65)
-			(end 2.1 1.26)
+			(start 3 -1.75)
+			(end -3 -1.75)
 			(stroke
-				(width 0.12)
+				(width 0.05)
 				(type solid)
 			)
-			(layer "F.SilkS")
+			(layer "F.CrtYd")
 		)
 		(fp_line
@@
 		)
 		(fp_line
-			(start -3 1.75)
-			(end 3 1.75)
+			(start 3 1.75)
+			(end 3 -1.75)
 			(stroke
 				(width 0.05)
@@
 		)
 		(fp_line
-			(start 3 -1.75)
-			(end -3 -1.75)
+			(start -3 1.75)
+			(end 3 1.75)
 			(stroke
 				(width 0.05)
@@
 		)
 		(fp_line
-			(start 3 1.75)
-			(end 3 -1.75)
+			(start 1.95 -1.5)
+			(end 1.95 1.5)
 			(stroke
-				(width 0.05)
+				(width 0.1)
 				(type solid)
 			)
-			(layer "F.CrtYd")
+			(layer "F.Fab")
 		)
 		(fp_line
@@
 			(layer "F.Fab")
 		)
-		(fp_line
-			(start 1.95 -1.5)
-			(end 1.95 1.5)
-			(stroke
-				(width 0.1)
-				(type solid)
-			)
-			(layer "F.Fab")
-		)
 		(fp_circle
 			(center 0 0)
@@
 		)
 		(pad "1" smd roundrect
-			(at -2.225 0)
+			(at -2.225 0 90)
 			(size 1.05 2)
 			(layers "F.Cu" "F.Mask" "F.Paste")
@@
 		)
 		(pad "2" smd roundrect
-			(at 2.225 0)
+			(at 2.225 0 90)
 			(size 1.05 2)
 			(layers "F.Cu" "F.Mask" "F.Paste")
@@
 	)
 	(segment
-		(start 110.75 110.75)
+		(start 111.5 110)
 		(end 110.360624 111.139376)
 		(width 0.2)
@@
 	)
 	(via
-		(at 110.75 110.75)
+		(at 111.5 110)
 		(size 0.6)
 		(drill 0.3)
@@
 	)
 	(via
-		(at 113.75 113.75)
-		(size 0.6)
-		(drill 0.3)
-		(layers "F.Cu" "B.Cu")
-		(free yes)
-		(net 2)
-	)
-	(via
 		(at 131.896 107.77)
 		(size 0.6)
@@
 	)
 	(segment
-		(start 114.34 112.24)
-		(end 114.6 112.5)
-		(width 0.2)
-		(layer "F.Cu")
-		(net 5)
-	)
-	(segment
 		(start 114.6 112.5)
 		(end 114.6 112)
@@
 	)
 	(segment
-		(start 112.75 112.24)
-		(end 114.34 112.24)
-		(width 0.2)
-		(layer "F.Cu")
-		(net 5)
-	)
-	(segment
 		(start 120.4585 104.5625)
 		(end 121.096 104.5625)
@@
 	)
 	(segment
-		(start 112.75 112.24)
-		(end 114.36 112.24)
-		(width 0.2)
-		(layer "F.Cu")
-		(net 5)
-	)
-	(segment
 		(start 114 110.73)
 		(end 113.95174 110.73)
@@
 	)
 	(segment
+		(start 114 110.73)
+		(end 113.01 110.73)
+		(width 0.3)
+		(layer "F.Cu")
+		(net 5)
+	)
+	(segment
 		(start 130.436 111.105686)
 		(end 130.436 111.5)
@@
 	)
 	(segment
-		(start 114.36 112.24)
-		(end 114.6 112)
-		(width 0.2)
-		(layer "F.Cu")
-		(net 5)
-	)
-	(segment
 		(start 118.92308 108.25)
 		(end 117.67308 109.5)
@@
 	)
 	(segment
+		(start 113.01 110.73)
+		(end 112.75 110.99)
+		(width 0.3)
+		(layer "F.Cu")
+		(net 5)
+	)
+	(segment
 		(start 121.297 105.651)
 		(end 121.297 104.7635)
@@
 	)
 	(segment
-		(start 108.51 119.75)
-		(end 107.25 119.75)
+		(start 111.5 113.5)
+		(end 111.5 112.01)
 		(width 0.2)
 		(layer "F.Cu")
@@
 	)
 	(segment
-		(start 112.75 115.51)
-		(end 108.51 119.75)
+		(start 118.253 112.4641)
+		(end 118.253 113.6859)
 		(width 0.2)
 		(layer "F.Cu")
-		(net 28)
+		(net 29)
 	)
 	(segment
-		(start 118.253 112.4641)
-		(end 118.253 113.6859)
+		(start 111.73 110.99)
+		(end 112.75 112.01)
+		(width 0.2)
+		(layer "F.Cu")
+		(net 29)
+	)
+	(segment
+		(start 111.5 110.99)
+		(end 111.73 110.99)
 		(width 0.2)
 		(layer "F.Cu")
@@
 	)
 	(segment
-		(start 114.55 115.25)
-		(end 114.6 115.2)
+		(start 113.75 112.5)
+		(end 113.26 112.01)
 		(width 0.2)
 		(layer "F.Cu")
@@
 	)
 	(segment
-		(start 112.75 113.26)
-		(end 112.75 114.49)
+		(start 114.55 115.25)
+		(end 114.6 115.2)
 		(width 0.2)
 		(layer "F.Cu")
@@
 	)
 	(segment
+		(start 113.75 114.35)
+		(end 113.75 112.5)
+		(width 0.2)
+		(layer "F.Cu")
+		(net 29)
+	)
+	(segment
 		(start 120.4585 110.8)
 		(end 120.45 110.8)
@@
 	)
 	(segment
-		(start 112.75 114.49)
-		(end 113.24 114.49)
+		(start 113.26 112.01)
+		(end 112.75 112.01)
 		(width 0.2)
 		(layer "F.Cu")
@@
 	)
 	(segment
-		(start 113.24 114.49)
-		(end 113.95 115.2)
-		(width 0.2)
-		(layer "F.Cu")
-		(net 29)
-	)
-	(segment
-		(start 113.95 115.2)
-		(end 114.6 115.2)
+		(start 114.6 115.2)
+		(end 113.75 114.35)
 		(width 0.2)
 		(layer "F.Cu")

Commit message: work
Parts:
- moved U8 0.57 mm to (116.2, 113.5)
Routing:
- net GND: track 71.8 -> 69.8 mm
- net /GPIO0: track 6.48 -> 5.35 mm
- net /QSPI_SD1: track 10.1 -> 9.31 mm
- net /QSPI_SS: track 17.1 -> 16.4 mm
- net /QSPI_SD2: track 7.77 -> 7.21 mm
- net /QSPI_SCLK: track 5.78 -> 5.24 mm
- net /QSPI_SD0: track 4.94 -> 4.41 mm

Commit message: work
Parts:
- moved R5 1.68 mm to (118.2, 102.5), turned to -90 degrees
- moved C9 0.27 mm to (117.0, 102.5), turned to 90 degrees
Routing:
- net GND: track 69.8 -> 81.5 mm, vias 24 -> 26
- net /SWD: track 24.4 -> 22.5 mm
- net +3V3: track 72.8 -> 74.3 mm
- net /SWCLK: track 21.4 -> 20.0 mm
- net /GPIO8: track 5.52 -> 4.62 mm
- net /VREG_AVDD: track 5.36 -> 4.62 mm
- net /ROW_D_5V: track 11.5 -> 10.8 mm
- net /GPIO11: track 5.64 -> 6.18 mm
