File: board/ioAmp200W.kicad_sch (KiCad schematic)
At the start: 32 parts, among them J1 USB_C_Receptacle_USB2.0_14P, J2 USB_C_Receptacle_USB2.0_14P, J4 SM03B-SRSS-TB, SW1 SW_Push, SW2 SW_Push, U1 RP2350_60QFN, Y1 ABM8-272-T3

Commit message: work
Parts:
- removed J1, J2: USB_C_Receptacle_USB2.0_14P, Connector_USB:USB_C_Receptacle_HRO_TYPE-C-31-M-12, symbol Connector:USB_C_Receptacle_USB2.0_14P
- added J1, J2: USB4105-GF-A-120, USB4105_GF_A_120:GCT_USB4105-GF-A-120, symbol USB4105-GF-A-120:USB4105-GF-A-120
- added U2: TPS26750SRSMR, TI2:VQFN32_RSM_TEX, symbol TI2:TPS26750SRSMR
- added U3: TPD4S480RUKR, TI:RUK0020B-MFG, symbol TI:TPD4S480RUKR
- added U4: ADAU1761BCPZ-RL, adau1761:CP-32-4_ADI, symbol adau1761:ADAU1761BCPZ-RL
Connections:
- net +5V: now also J1.A4_B9 (VBUS), J1.B4_A9 (VBUS__1)
- net GND: now also J1.A1_B12 (GND), J1.B1_A12 (GND__1), J1.SH1 (SHELL_GND), J1.SH2 (SHELL_GND__1), J1.SH3 (SHELL_GND__2), J1.SH4 (SHELL_GND__3), J2.A1_B12 (GND), J2.B1_A12 (GND__1), J2.SH1 (SHELL_GND), J2.SH2 (SHELL_GND__1), J2.SH3 (SHELL_GND__2), J2.SH4 (SHELL_GND__3); no longer R3.1, R4.1
- net USB_D+: now also J1.A6 (DP1), J1.B6 (DP2)
- net USB_D-: now also J1.A7 (DN1), J1.B7 (DN2)
- net at R4.2: now also J1.A5 (CC1)
- net at R3.2: now also J1.B5 (CC2)
- no-connect marks 5 -> 7
Other:
- moved on the sheet: C10, C11, C12, C13, C14, C15, C16, C17, C18, C2, C3, C4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

Commit message: work
Parts:
- added H1, H2, H3, H4: MountingHole_Pad_MP, MountingHole:MountingHole_2.2mm_M2_ISO7380_Pad_TopBottom, symbol Mechanical:MountingHole_Pad_MP
- added J3: AudioJack3_Ground, Connector_Audio:Jack_3.5mm_PJ320D_Horizontal, symbol Connector_Audio:AudioJack3_Ground
- added J5, J6: Conn_01x02_Socket, Connector_AMASS:AMASS_XT30U-F_1x02_P5.0mm_Vertical, symbol Connector:Conn_01x02_Socket
- renumbered J1 to USB_DATA1, J2 to USB_POWER1
Connections:
- net GND: now also H1.MP, H2.MP, H3.MP, H4.MP
Other:
- note added: "OUTPUT CONNECTORS"

Commit message: work
Parts:
- renumbered J6 to L_OUT1, J5 to R_OUT1, J3 to TRS1
Other:
- moved on the sheet: L_OUT1, R_OUT1
Changed lines of the file:
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@@
 		(dnp no)
 		(fields_autoplaced yes)
-		(property "Reference" "J3"
+		(property "Reference" "TRS1"
 			(at 93.345 449.58 0)
 			(effects
@@
 			(project ""
 				(path "/4f3b51aa-8e6e-4521-ad6c-a7e6e194e2a4"
-					(reference "J3")
+					(reference "TRS1")
 					(unit 1)
 				)
@@
 	(symbol
 		(lib_id "Connector:Conn_01x02_Socket")
-		(at 645.16 440.69 0)
+		(at 673.1 439.42 0)
 		(unit 1)
 		(exclude_from_sim no)
@@
 		(dnp no)
 		(fields_autoplaced yes)
-		(property "Reference" "J5"
-			(at 646.43 440.6899 0)
+		(property "Reference" "R_OUT1"
+			(at 674.37 439.4199 0)
 			(effects
 				(font
@@
 		)
 		(property "Value" "Conn_01x02_Socket"
-			(at 646.43 443.2299 0)
+			(at 674.37 441.9599 0)
 			(effects
 				(font
@@
 		)
 		(property "Footprint" "Connector_AMASS:AMASS_XT30U-F_1x02_P5.0mm_Vertical"
-			(at 645.16 440.69 0)
+			(at 673.1 439.42 0)
 			(effects
 				(font
@@
 		)
 		(property "Datasheet" "~"
-			(at 645.16 440.69 0)
+			(at 673.1 439.42 0)
 			(effects
 				(font
@@
 		)
 		(property "Description" "Generic connector, single row, 01x02, script generated"
-			(at 645.16 440.69 0)
+			(at 673.1 439.42 0)
 			(effects
 				(font
@@
 			(project ""
 				(path "/4f3b51aa-8e6e-4521-ad6c-a7e6e194e2a4"
-					(reference "J5")
+					(reference "R_OUT1")
 					(unit 1)
 				)
@@
 	(symbol
 		(lib_id "Connector:Conn_01x02_Socket")
-		(at 675.64 440.69 0)
+		(at 643.89 439.42 0)
 		(unit 1)
 		(exclude_from_sim no)
@@
 		(dnp no)
 		(fields_autoplaced yes)
-		(property "Reference" "J6"
-			(at 676.91 440.6899 0)
+		(property "Reference" "L_OUT1"
+			(at 645.16 439.4199 0)
 			(effects
 				(font
@@
 		)
 		(property "Value" "Conn_01x02_Socket"
-			(at 676.91 443.2299 0)
+			(at 645.16 441.9599 0)
 			(effects
 				(font
@@
 		)
 		(property "Footprint" "Connector_AMASS:AMASS_XT30U-F_1x02_P5.0mm_Vertical"
-			(at 675.64 440.69 0)
+			(at 643.89 439.42 0)
 			(effects
 				(font
@@
 		)
 		(property "Datasheet" "~"
-			(at 675.64 440.69 0)
+			(at 643.89 439.42 0)
 			(effects
 				(font
@@
 		)
 		(property "Description" "Generic connector, single row, 01x02, script generated"
-			(at 675.64 440.69 0)
+			(at 643.89 439.42 0)
 			(effects
 				(font
@@
 			(project "ioAmp200W"
 				(path "/4f3b51aa-8e6e-4521-ad6c-a7e6e194e2a4"
-					(reference "J6")
-					(unit 1)
-				)
+					(reference "L_OUT1")
+					(unit 1)
+				)

Commit message: work
Parts:
- removed H1, H2, H3, H4: MountingHole_Pad_MP, MountingHole:MountingHole_2.2mm_M2_ISO7380_Pad_TopBottom, symbol Mechanical:MountingHole_Pad_MP
- added H1, H2, H3, H4: MountingHole, MountingHole:MountingHole_2.1mm, symbol Mechanical:MountingHole
Other:
- note added: "Designed by Isaac Olson"
- note removed: "Designed at Audio and Arduino Club Isaac Olson"

Commit message: work
Connections:
- net GPIO26_ADC0 is gone; now on net GND: U1.40 (GPIO26_ADC0)
- net GPIO27_ADC1 is gone; now on net GND: U1.41 (GPIO27_ADC1)
- net GPIO28_ADC2 is gone; now on net GND: U1.42 (GPIO28_ADC2)
- net GPIO29_ADC3 is gone; now on net GND: U1.43 (GPIO29_ADC3)
Changed lines of the file:
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@@
 	)
 	(junction
+		(at 276.86 302.26)
+		(diameter 0)
+		(color 0 0 0 0)
+	)
+	(junction
 		(at 289.56 186.69)
 		(diameter 0)
@@
 	)
 	(junction
+		(at 276.86 297.18)
+		(diameter 0)
+		(color 0 0 0 0)
+	)
+	(junction
 		(at 175.26 185.42)
 		(diameter 0)
@@
 	)
 	(junction
+		(at 276.86 299.72)
+		(diameter 0)
+		(color 0 0 0 0)
+	)
+	(junction
 		(at 323.85 186.69)
 		(diameter 0)
@@
 	(wire
 		(pts
+			(xy 276.86 297.18) (xy 276.86 299.72)
+		)
+		(stroke
+			(width 0)
+			(type default)
+		)
+	)
+	(wire
+		(pts
 			(xy 93.98 292.1) (xy 107.95 292.1)
 		)
@@
 	(wire
 		(pts
+			(xy 276.86 299.72) (xy 276.86 302.26)
+		)
+		(stroke
+			(width 0)
+			(type default)
+		)
+	)
+	(wire
+		(pts
 			(xy 261.62 289.56) (xy 276.86 289.56)
 		)
@@
 	(wire
 		(pts
+			(xy 276.86 302.26) (xy 276.86 304.8)
+		)
+		(stroke
+			(width 0)
+			(type default)
+		)
+	)
+	(wire
+		(pts
 			(xy 300.99 184.15) (xy 300.99 186.69)
 		)
@@
 	(wire
 		(pts
+			(xy 276.86 294.64) (xy 276.86 297.18)
+		)
+		(stroke
+			(width 0)
+			(type default)
+		)
+	)
+	(wire
+		(pts
 			(xy 87.63 287.02) (xy 88.9 287.02)
 		)
@@
 		)
 	)
-	(label "GPIO26_ADC0"
-		(at 276.86 294.64 180)
-		(effects
-			(font
-				(size 1.27 1.27)
-			)
-			(justify right bottom)
-		)
-	)
 	(label "USB_D-"
 		(at 435.61 236.22 180)
@@
 		)
 	)
-	(label "GPIO27_ADC1"
-		(at 276.86 297.18 180)
-		(effects
-			(font
-				(size 1.27 1.27)
-			)
-			(justify right bottom)
-		)
-	)
 	(label "GPIO23"
 		(at 276.86 284.48 180)
@@
 		)
 	)
-	(label "GPIO28_ADC2"
-		(at 276.86 299.72 180)
-		(effects
-			(font
-				(size 1.27 1.27)
-			)
-			(justify right bottom)
-		)
-	)
 	(label "GPIO21"
 		(at 276.86 279.4 180)
@@
 		)
 	)
-	(label "GPIO29_ADC3"
-		(at 276.86 302.26 180)
-		(effects
-			(font
-				(size 1.27 1.27)
-			)
-			(justify right bottom)
-		)
-	)
 	(label "RUN"
 		(at 184.15 279.4 0)
@@
 					(unit 1)
 				)
+			)
+		)
+	)
+	(symbol
+		(lib_id "power:GND")
+		(at 276.86 304.8 0)
+		(unit 1)
+		(exclude_from_sim no)
+		(in_bom yes)
+		(on_board yes)
+		(dnp no)
+		(fields_autoplaced yes)
+		(property "Reference" "#PWR07"
+			(at 276.86 311.15 0)
+			(effects
+				(font
+					(size 1.27 1.27)
+				)
+				(hide yes)
+			)
+		)
+		(property "Value" "GND"
+			(at 276.86 309.88 0)
+			(effects
+				(font
+					(size 1.27 1.27)
+				)
+			)
+		)
+		(property "Footprint" ""
+			(at 276.86 304.8 0)
+			(effects
+				(font
+					(size 1.27 1.27)
+				)
+				(hide yes)
+			)
+		)
+		(property "Datasheet" ""
+			(at 276.86 304.8 0)
+			(effects
+				(font
+					(size 1.27 1.27)
+				)
+				(hide yes)
+			)
+		)
+		(property "Description" "Power symbol creates a global label with name \"GND\" , ground"
+			(at 276.86 304.8 0)
+			(effects
+				(font
+					(size 1.27 1.27)
+				)
+				(hide yes)
+			)
+		)
+		(pin "1"
+		)
+		(instances
+			(project ""
+				(path "/4f3b51aa-8e6e-4521-ad6c-a7e6e194e2a4"
+					(reference "#PWR07")
+					(unit 1)
+				)

Commit message: switch_dsp
Parts:
- removed U4: ADAU1761BCPZ-RL, adau1761:CP-32-4_ADI, symbol adau1761:ADAU1761BCPZ-RL
- added U4: TLV320AIC3204IRHBR, TLV320AIC3204IRHBR:QFN50P500X500X100-33N, symbol TLV320AIC3204IRHBR:TLV320AIC3204IRHBR
Changed lines of the file:
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@@
-	)
-	(symbol
-		(lib_id "adau1761:ADAU1761BCPZ-RL")
-		(at 152.4 434.34 0)
-		(unit 1)
-		(exclude_from_sim no)
-		(in_bom yes)
-		(on_board yes)
-		(dnp no)
-		(fields_autoplaced yes)
-		(property "Reference" "U4"
-			(at 195.58 424.18 0)
-			(effects
-				(font
-					(size 1.524 1.524)
-				)
-			)
-		)
-		(property "Value" "ADAU1761BCPZ-RL"
-			(at 195.58 426.72 0)
-			(effects
-				(font
-					(size 1.524 1.524)
-				)
-			)
-		)
-		(property "Footprint" "adau1761:CP-32-4_ADI"
-			(at 152.4 434.34 0)
-			(effects
-				(font
-					(size 1.27 1.27)
-					(italic yes)
-				)
-				(hide yes)
-			)
-		)
-		(property "Datasheet" "https://www.analog.com/media/en/technical-documentation/data-sheets/ADAU1761.pdf"
-			(at 152.4 434.34 0)
-			(effects
-				(font
-					(size 1.27 1.27)
-					(italic yes)
-				)
-				(hide yes)
-			)
-		)
-		(property "Description" ""
-			(at 152.4 434.34 0)
-			(effects
-				(font
-					(size 1.27 1.27)
-				)
-				(hide yes)
-			)
-		)
-		(pin "17"
-		)
-		(pin "18"
-		)
-		(pin "19"
-		)
-		(pin "20"
-		)
-		(pin "21"
-		)
-		(pin "22"
-		)
-		(pin "23"
-		)
-		(pin "24"
-		)
-		(pin "25"
-		)
-		(pin "6"
-		)
-		(pin "5"
-		)
-		(pin "4"
-		)
-		(pin "3"
-		)
-		(pin "2"
-		)
-		(pin "1"
-		)
-		(pin "11"
-		)
-		(pin "10"
-		)
-		(pin "9"
-		)
-		(pin "8"
-		)
-		(pin "7"
-		)
-		(pin "12"
-		)
-		(pin "13"
-		)
-		(pin "14"
-		)
-		(pin "15"
-		)
-		(pin "16"
-		)
-		(pin "26"
-		)
-		(pin "27"
-		)
-		(pin "28"
-		)
-		(pin "29"
-		)
-		(pin "30"
-		)
-		(pin "31"
-		)
-		(pin "32"
-		)
-		(pin "33"
-		)
-		(instances
-			(project ""
-				(path "/4f3b51aa-8e6e-4521-ad6c-a7e6e194e2a4"
-					(reference "U4")
-					(unit 1)
-				)
-			)
-		)
 	)
 	(symbol
@@
 					(unit 1)
 				)
+			)
+		)
+	)
+	(symbol
+		(lib_id "TLV320AIC3204IRHBR:TLV320AIC3204IRHBR")
+		(at 181.61 454.66 0)
+		(unit 1)
+		(exclude_from_sim no)
+		(in_bom yes)
+		(on_board yes)
+		(dnp no)
+		(fields_autoplaced yes)
+		(property "Reference" "U4"
+			(at 181.61 411.48 0)
+			(effects
+				(font
+					(size 1.27 1.27)
+				)
+			)
+		)
+		(property "Value" "TLV320AIC3204IRHBR"
+			(at 181.61 414.02 0)
+			(effects
+				(font
+					(size 1.27 1.27)
+				)
+			)
+		)
+		(property "Footprint" "TLV320AIC3204IRHBR:QFN50P500X500X100-33N"
+			(at 181.61 454.66 0)
+			(effects
+				(font
+					(size 1.27 1.27)
+				)
+				(justify bottom)
+				(hide yes)
+			)
+		)
+		(property "Datasheet" ""
+			(at 181.61 454.66 0)
+			(effects
+				(font
+					(size 1.27 1.27)
+				)
+				(hide yes)
+			)
+		)
+		(property "Description" ""
+			(at 181.61 454.66 0)
+			(effects
+				(font
+					(size 1.27 1.27)
+				)
+				(hide yes)
+			)
+		)
+		(property "PARTREV" "E"
+			(at 181.61 454.66 0)
+			(effects
+				(font
+					(size 1.27 1.27)
+				)
+				(justify bottom)
+				(hide yes)
+			)
+		)
+		(property "STANDARD" "IPC-7351B"
+			(at 181.61 454.66 0)
+			(effects
+				(font
+					(size 1.27 1.27)
+				)
+				(justify bottom)
+				(hide yes)
+			)
+		)
+		(property "MAXIMUM_PACKAGE_HEIGHT" "1.0mm"
+			(at 181.61 454.66 0)
+			(effects
+				(font
+					(size 1.27 1.27)
+				)
+				(justify bottom)
+				(hide yes)
+			)
+		)
+		(property "MANUFACTURER" "Texas Instruments"
+			(at 181.61 454.66 0)
+			(effects
+				(font
+					(size 1.27 1.27)
+				)
+				(justify bottom)
+				(hide yes)
+			)
+		)
+		(pin "32"
+		)
+		(pin "13"
+		)
+		(pin "11"
+		)
+		(pin "8"
+		)
+		(pin "10"
+		)
+		(pin "30"
+		)
+		(pin "9"
+		)
+		(pin "29"
+		)
+		(pin "24"
+		)
+		(pin "26"
+		)
+		(pin "31"
+		)
+		(pin "15"
+		)
+		(pin "12"
+		)
+		(pin "5"
+		)
+		(pin "21"
+		)
+		(pin "20"
+		)
+		(pin "19"
+		)
+		(pin "6"
+		)
+		(pin "16"
+		)
+		(pin "18"
+		)
+		(pin "14"
+		)
+		(pin "33"
+		)
+		(pin "1"
+		)
+		(pin "27"
+		)
+		(pin "28"
+		)
+		(pin "25"
+		)
+		(pin "2"
+		)
+		(pin "17"
+		)
+		(pin "3"
+		)
+		(pin "23"
+		)
+		(pin "7"
+		)
+		(pin "4"
+		)
+		(pin "22"
+		)
+		(instances
+			(project ""
+				(path "/4f3b51aa-8e6e-4521-ad6c-a7e6e194e2a4"
+					(reference "U4")
+					(unit 1)
+				)

Commit message: work
Parts:
- U4: value TLV320AIC3204IRHBR -> TLV320AIC3256
Connections:
- net +3V3: now also U2.1 (LDO_3V3)
- net GND: now also TRS1.G, U4.17 (AVSS), U4.28 (DVSS), U4.33 (EP), U4.7 (IOVSS)
Other:
- moved on the sheet: C10, C11, C12, C13, C14, C15, C16, C17, C18, C2, C3, C4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

Commit message: work
Parts:
- added U5: MA5332MS, Library:IFX-PG-IQFN-42-1-V, symbol Amplifier_Buffer:MA5332MS
Connections:
- no-connect marks 7 -> 8
Other:
- moved on the sheet: L_OUT1, R_OUT1
Changed lines of the file:
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@@
 	(text "OUTPUT CONNECTORS"
 		(exclude_from_sim no)
-		(at 518.922 428.498 0)
+		(at 526.288 520.7 0)
 		(effects
 			(font
@@
 		(exclude_from_sim no)
 		(at 375.92 248.92 0)
-		(size 295.91 210.82)
+		(size 295.91 283.21)
 		(margins 0.9525 0.9525 0.9525 0.9525)
 		(stroke
@@
 		)
 	)
-	(text_box "POWER MANAGEMENT"
+	(text_box "POWER MANAGEMENT SYSTEM"
 		(exclude_from_sim no)
 		(at 25.4 248.92 0)
@@
 		)
 	)
-	(text_box "DSP"
+	(text_box "CODEC / DSP"
 		(exclude_from_sim no)
 		(at 25.4 368.3 0)
@@
 	)
 	(no_connect
+		(at 535.94 369.57)
+	)
+	(no_connect
 		(at 394.97 125.73)
 	)
@@
 	(symbol
 		(lib_id "Connector:Conn_01x02_Socket")
-		(at 528.32 436.88 0)
+		(at 534.67 509.27 0)
 		(unit 1)
 		(exclude_from_sim no)
@@
 		(fields_autoplaced yes)
 		(property "Reference" "R_OUT1"
-			(at 529.59 436.8799 0)
+			(at 535.94 509.2699 0)
 			(effects
 				(font
@@
 		)
 		(property "Value" "Conn_01x02_Socket"
-			(at 529.59 439.4199 0)
+			(at 535.94 511.8099 0)
 			(effects
 				(font
@@
 		)
 		(property "Footprint" "Connector_AMASS:AMASS_XT30U-F_1x02_P5.0mm_Vertical"
-			(at 528.32 436.88 0)
+			(at 534.67 509.27 0)
 			(effects
 				(font
@@
 		)
 		(property "Datasheet" "~"
-			(at 528.32 436.88 0)
+			(at 534.67 509.27 0)
 			(effects
 				(font
@@
 		)
 		(property "Description" "Generic connector, single row, 01x02, script generated"
-			(at 528.32 436.88 0)
+			(at 534.67 509.27 0)
 			(effects
 				(font
@@
 	(symbol
 		(lib_id "Connector:Conn_01x02_Socket")
-		(at 499.11 436.88 0)
+		(at 500.38 509.27 0)
 		(unit 1)
 		(exclude_from_sim no)
@@
 		(fields_autoplaced yes)
 		(property "Reference" "L_OUT1"
-			(at 500.38 436.8799 0)
+			(at 501.65 509.2699 0)
 			(effects
 				(font
@@
 		)
 		(property "Value" "Conn_01x02_Socket"
-			(at 500.38 439.4199 0)
+			(at 501.65 511.8099 0)
 			(effects
 				(font
@@
 		)
 		(property "Footprint" "Connector_AMASS:AMASS_XT30U-F_1x02_P5.0mm_Vertical"
-			(at 499.11 436.88 0)
+			(at 500.38 509.27 0)
 			(effects
 				(font
@@
 		)
 		(property "Datasheet" "~"
-			(at 499.11 436.88 0)
+			(at 500.38 509.27 0)
 			(effects
 				(font
@@
 		)
 		(property "Description" "Generic connector, single row, 01x02, script generated"
-			(at 499.11 436.88 0)
+			(at 500.38 509.27 0)
 			(effects
 				(font
@@
 					(unit 1)
 				)
+			)
+		)
+	)
+	(symbol
+		(lib_id "Amplifier_Buffer:MA5332MS")
+		(at 508 308.61 0)
+		(unit 1)
+		(exclude_from_sim no)
+		(in_bom yes)
+		(on_board yes)
+		(dnp no)
+		(fields_autoplaced yes)
+		(property "Reference" "U5"
+			(at 519.43 302.26 0)
+			(effects
+				(font
+					(size 1.8288 1.8288)
+				)
+			)
+		)
+		(property "Value" "MA5332MS"
+			(at 519.43 306.07 0)
+			(effects
+				(font
+					(size 1.8288 1.8288)
+				)
+			)
+		)
+		(property "Footprint" "Library:IFX-PG-IQFN-42-1-V"
+			(at 508 308.61 0)
+			(effects
+				(font
+					(size 1.27 1.27)
+				)
+				(hide yes)
+			)
+		)
+		(property "Datasheet" ""
+			(at 508 308.61 0)
+			(effects
+				(font
+					(size 1.27 1.27)
+				)
+				(hide yes)
+			)
+		)
+		(property "Description" "200W Stereo, Integrated Class D Amplifier"
+			(at 508 308.61 0)
+			(effects
+				(font
+					(size 1.27 1.27)
+				)
+				(hide yes)
+			)
+		)
+		(property "Manufacturer Order Number" "MA5332MS"
+			(at 492.252 321.31 0)
+			(effects
+				(font
+					(size 1.8288 1.8288)
+				)
+				(justify left bottom)
+				(hide yes)
+			)
+		)
+		(property "PackageReference" "PG-IQFN-42-1"
+			(at 502.412 346.71 0)
+			(effects
+				(font
+					(size 1.8288 1.8288)
+				)
+				(justify left bottom)
+				(hide yes)
+			)
+		)
+		(property "Manufacturer" "Infineon Technologies"
+			(at 502.412 377.19 0)
+			(effects
+				(font
+					(size 1.8288 1.8288)
+				)
+				(justify left bottom)
+				(hide yes)
+			)
+		)
+		(pin "20"
+		)
+		(pin "18"
+		)
+		(pin "19"
+		)
+		(pin "22"
+		)
+		(pin "17"
+		)
+		(pin "15"
+		)
+		(pin "21"
+		)
+		(pin "23"
+		)
+		(pin "24"
+		)
+		(pin "25"
+		)
+		(pin "16"
+		)
+		(pin "26"
+		)
+		(pin "28"
+		)
+		(pin "14"
+		)
+		(pin "27"
+		)
+		(pin "12"
+		)
+		(pin "5"
+		)
+		(pin "6"
+		)
+		(pin "1"
+		)
+		(pin "7"
+		)
+		(pin "3"
+		)
+		(pin "2"
+		)
+		(pin "13"
+		)
+		(pin "9"
+		)
+		(pin "11"
+		)
+		(pin "8"
+		)
+		(pin "10"
+		)
+		(pin "4"
+		)
+		(instances
+			(project ""
+				(path "/4f3b51aa-8e6e-4521-ad6c-a7e6e194e2a4"
+					(reference "U5")
+					(unit 1)
+				)
