File: board/ioAmp200W.kicad_sch (KiCad schematic)
At the start: 139 parts, among them J1 USB4105-GF-A-120, J2 USB4105-GF-A-120, J3 Speaker_Out, J4 SM03B-SRSS-TB, SW1 SW_Push, U1 RP2350_60QFN, U10 TPS7A1601DRBR, U2 TPS26750SRSMR, U3 TPD4S480RUKR, U4 TLV320AIC3254IRHBT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

Commit message: dcdc
Connections:
- net +10V: now also U10.1 (OUT)
- net VBUS: now also U10.5 (EN), U10.8 (IN)
- net at C64.2: now also U4.13 (IN1_L); no longer U4.20 (IN3_L)
- net at U4.14 (IN1_R): now also C65.2
- net at U4.21 (IN3_R): no longer C65.2
- no-connect marks 11 -> 12
Other:
- moved on the sheet: U10
Changed lines of the file:
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@@
 	)
 	(junction
-		(at 166.37 308.61)
-		(diameter 0)
-		(color 0 0 0 0)
-	)
-	(junction
 		(at 147.32 93.98)
 		(diameter 0)
@@
 	)
 	(junction
+		(at 595.63 427.99)
+		(diameter 0)
+		(color 0 0 0 0)
+	)
+	(junction
 		(at 91.44 468.63)
 		(diameter 0)
@@
 	)
 	(no_connect
-		(at 179.07 299.72)
-	)
-	(no_connect
 		(at 435.61 128.27)
 	)
@@
 	)
 	(no_connect
-		(at 596.9 429.26)
+		(at 638.81 128.27)
 	)
 	(no_connect
-		(at 638.81 128.27)
+		(at 229.87 292.1)
 	)
 	(no_connect
@@
 	)
 	(no_connect
+		(at 229.87 294.64)
+	)
+	(no_connect
 		(at 638.81 125.73)
 	)
@@
 	)
 	(no_connect
-		(at 179.07 302.26)
+		(at 179.07 312.42)
+	)
+	(no_connect
+		(at 179.07 309.88)
 	)
 	(wire
@@
 	(wire
 		(pts
-			(xy 158.75 308.61) (xy 157.48 308.61)
-		)
-		(stroke
-			(width 0)
-			(type default)
-		)
-	)
-	(wire
-		(pts
 			(xy 229.87 350.52) (xy 229.87 354.33)
 		)
@@
 	(wire
 		(pts
-			(xy 166.37 308.61) (xy 165.1 308.61)
-		)
-		(stroke
-			(width 0)
-			(type default)
-		)
-	)
-	(wire
-		(pts
 			(xy 554.99 283.21) (xy 576.58 283.21)
 		)
@@
 	(wire
 		(pts
-			(xy 167.64 303.53) (xy 167.64 309.88)
-		)
-		(stroke
-			(width 0)
-			(type default)
-		)
-	)
-	(wire
-		(pts
 			(xy 628.65 107.95) (xy 638.81 107.95)
 		)
@@
 	(wire
 		(pts
-			(xy 179.07 309.88) (xy 167.64 309.88)
-		)
-		(stroke
-			(width 0)
-			(type default)
-		)
-	)
-	(wire
-		(pts
 			(xy 101.6 450.85) (xy 91.44 450.85)
 		)
@@
 	(wire
 		(pts
-			(xy 166.37 303.53) (xy 167.64 303.53)
+			(xy 166.37 303.53) (xy 168.91 303.53)
 		)
 		(stroke
@@
 	(wire
 		(pts
+			(xy 168.91 299.72) (xy 168.91 303.53)
+		)
+		(stroke
+			(width 0)
+			(type default)
+		)
+	)
+	(wire
+		(pts
 			(xy 612.14 372.11) (xy 604.52 372.11)
 		)
@@
 	(wire
 		(pts
+			(xy 179.07 302.26) (xy 171.45 302.26)
+		)
+		(stroke
+			(width 0)
+			(type default)
+		)
+	)
+	(wire
+		(pts
 			(xy 193.04 491.49) (xy 193.04 494.03)
 		)
@@
 	(wire
 		(pts
-			(xy 127 307.34) (xy 157.48 307.34)
+			(xy 127 307.34) (xy 158.75 307.34)
 		)
 		(stroke
@@
 	(wire
 		(pts
-			(xy 157.48 308.61) (xy 157.48 307.34)
+			(xy 158.75 308.61) (xy 158.75 307.34)
 		)
 		(stroke
@@
 	(wire
 		(pts
-			(xy 158.75 303.53) (xy 157.48 303.53)
-		)
-		(stroke
-			(width 0)
-			(type default)
-		)
-	)
-	(wire
-		(pts
 			(xy 631.19 361.95) (xy 624.84 361.95)
 		)
@@
 	(wire
 		(pts
-			(xy 179.07 312.42) (xy 166.37 312.42)
-		)
-		(stroke
-			(width 0)
-			(type default)
-		)
-	)
-	(wire
-		(pts
 			(xy 269.24 138.43) (xy 284.48 138.43)
 		)
@@
 	(wire
 		(pts
-			(xy 166.37 308.61) (xy 166.37 312.42)
-		)
-		(stroke
-			(width 0)
-			(type default)
-		)
-	)
-	(wire
-		(pts
 			(xy 148.59 314.96) (xy 158.75 314.96)
 		)
@@
 	(wire
 		(pts
+			(xy 554.99 427.99) (xy 554.99 412.75)
+		)
+		(stroke
+			(width 0)
+			(type default)
+		)
+	)
+	(wire
+		(pts
 			(xy 137.16 314.96) (xy 148.59 314.96)
 		)
@@
 	(wire
 		(pts
+			(xy 595.63 427.99) (xy 595.63 433.07)
+		)
+		(stroke
+			(width 0)
+			(type default)
+		)
+	)
+	(wire
+		(pts
 			(xy 342.9 66.04) (xy 342.9 64.77)
 		)
@@
 	(wire
 		(pts
+			(xy 595.63 412.75) (xy 591.82 412.75)
+		)
+		(stroke
+			(width 0)
+			(type default)
+		)
+	)
+	(wire
+		(pts
 			(xy 91.44 463.55) (xy 91.44 466.09)
 		)
@@
 	(wire
 		(pts
-			(xy 157.48 304.8) (xy 127 304.8)
+			(xy 158.75 304.8) (xy 127 304.8)
 		)
 		(stroke
@@
 	(wire
 		(pts
+			(xy 171.45 302.26) (xy 171.45 308.61)
+		)
+		(stroke
+			(width 0)
+			(type default)
+		)
+	)
+	(wire
+		(pts
 			(xy 167.005 139.7) (xy 167.005 142.24)
 		)
@@
 	(wire
 		(pts
+			(xy 179.07 299.72) (xy 168.91 299.72)
+		)
+		(stroke
+			(width 0)
+			(type default)
+		)
+	)
+	(wire
+		(pts
 			(xy 389.89 295.91) (xy 389.89 312.42)
 		)
@@
 	(wire
 		(pts
+			(xy 595.63 412.75) (xy 595.63 427.99)
+		)
+		(stroke
+			(width 0)
+			(type default)
+		)
+	)
+	(wire
+		(pts
 			(xy 269.24 133.35) (xy 284.48 133.35)
 		)
@@
 	(wire
 		(pts
+			(xy 554.99 412.75) (xy 558.8 412.75)
+		)
+		(stroke
+			(width 0)
+			(type default)
+		)
+	)
+	(wire
+		(pts
 			(xy 567.69 325.12) (xy 589.28 325.12)
 		)
@@
 	(wire
 		(pts
-			(xy 157.48 303.53) (xy 157.48 304.8)
+			(xy 158.75 303.53) (xy 158.75 304.8)
 		)
 		(stroke
@@
 	(wire
 		(pts
+			(xy 166.37 308.61) (xy 171.45 308.61)
+		)
+		(stroke
+			(width 0)
+			(type default)
+		)
+	)
+	(wire
+		(pts
 			(xy 377.19 321.31) (xy 396.24 321.31)
 		)
@@
 	(symbol
 		(lib_id "TPS7A:TPS7A1601DRBR")
-		(at 576.58 444.5 0)
+		(at 575.31 440.69 0)
 		(mirror y)
 		(unit 1)
@@
 		(dnp no)
 		(property "Reference" "U10"
-			(at 576.58 467.36 0)
+			(at 575.31 463.55 0)
 			(effects
 				(font
@@
 		)
 		(property "Value" "TPS7A1601DRBR"
-			(at 576.58 464.82 0)
+			(at 575.31 461.01 0)
 			(effects
 				(font
@@
 		)
 		(property "Footprint" "TPS26750SRSMR:VQFN32_RSM_TEX"
-			(at 576.58 444.5 0)
+			(at 575.31 440.69 0)
 			(effects
 				(font
@@
 		)
 		(property "Datasheet" "https://www.ti.com/lit/gpn/tps7a16"
-			(at 576.58 444.5 0)
+			(at 575.31 440.69 0)
 			(effects
 				(font
@@
 		)
 		(property "Description" ""
-			(at 576.58 444.5 0)
+			(at 575.31 440.69 0)
 			(effects
 				(font

Commit message: dcdc
Parts:
- added U11: LM76005QRNPRQ1, LM76005:RNP0030A, symbol LM76005:LM76005QRNPRQ1
Connections:
- no-connect marks 12 -> 19
Changed lines of the file:
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@@
 	)
 	(no_connect
+		(at 447.04 486.41)
+	)
+	(no_connect
+		(at 447.04 491.49)
+	)
+	(no_connect
 		(at 435.61 128.27)
 	)
@@
 	)
 	(no_connect
+		(at 447.04 481.33)
+	)
+	(no_connect
+		(at 447.04 496.57)
+	)
+	(no_connect
 		(at 638.81 128.27)
 	)
 	(no_connect
+		(at 447.04 488.95)
+	)
+	(no_connect
 		(at 229.87 292.1)
 	)
 	(no_connect
+		(at 447.04 494.03)
+	)
+	(no_connect
 		(at 394.97 125.73)
 	)
@@
 	)
 	(no_connect
+		(at 447.04 483.87)
+	)
+	(no_connect
 		(at 179.07 312.42)
 	)
@@
 					(unit 1)
 				)
+			)
+		)
+	)
+	(symbol
+		(lib_id "LM76005:LM76005QRNPRQ1")
+		(at 464.82 471.17 0)
+		(unit 1)
+		(exclude_from_sim no)
+		(in_bom yes)
+		(on_board yes)
+		(dnp no)
+		(fields_autoplaced yes)
+		(property "Reference" "U11"
+			(at 464.82 430.53 0)
+			(effects
+				(font
+					(size 1.524 1.524)
+				)
+			)
+		)
+		(property "Value" "LM76005QRNPRQ1"
+			(at 464.82 433.07 0)
+			(effects
+				(font
+					(size 1.524 1.524)
+				)
+			)
+		)
+		(property "Footprint" "LM76005:RNP0030A"
+			(at 464.82 471.17 0)
+			(effects
+				(font
+					(size 1.27 1.27)
+					(italic yes)
+				)
+				(hide yes)
+			)
+		)
+		(property "Datasheet" "https://www.ti.com/lit/gpn/lm76005-q1"
+			(at 464.82 471.17 0)
+			(effects
+				(font
+					(size 1.27 1.27)
+					(italic yes)
+				)
+				(hide yes)
+			)
+		)
+		(property "Description" ""
+			(at 464.82 471.17 0)
+			(effects
+				(font
+					(size 1.27 1.27)
+				)
+				(hide yes)
+			)
+		)
+		(pin "20"
+		)
+		(pin "8"
+		)
+		(pin "21"
+		)
+		(pin "22"
+		)
+		(pin "18"
+		)
+		(pin "16"
+		)
+		(pin "11"
+		)
+		(pin "10"
+		)
+		(pin "17"
+		)
+		(pin "7"
+		)
+		(pin "19"
+		)
+		(pin "23"
+		)
+		(pin "27"
+		)
+		(pin "28"
+		)
+		(pin "29"
+		)
+		(pin "30"
+		)
+		(pin "1"
+		)
+		(pin "2"
+		)
+		(pin "3"
+		)
+		(pin "4"
+		)
+		(pin "5"
+		)
+		(pin "6"
+		)
+		(pin "9"
+		)
+		(pin "12"
+		)
+		(pin "13"
+		)
+		(pin "14"
+		)
+		(pin "31"
+		)
+		(pin "26"
+		)
+		(pin "25"
+		)
+		(pin "24"
+		)
+		(pin "15"
+		)
+		(instances
+			(project ""
+				(path "/4f3b51aa-8e6e-4521-ad6c-a7e6e194e2a4"
+					(reference "U11")
+					(unit 1)
+				)

Commit message: dcdc
Parts:
- removed R3, R4: 5.1k, Resistor_SMD:R_0402_1005Metric, symbol Device:R
- added U12: TLV75733PDRVR, TLV75733PDRVR:DRV0006A_NV, symbol TLV75733PDRVR:TLV75733PDRVR
Connections:
- net +3V3: now also U12.1 (OUT)
- net EPR_SBU1: now also U3.15 (SBU1)
- net EPR_SBU2: now also U3.14 (SBU2)
- net GND: now also U10.4 (GND), U10.9 (PAD), U12.3 (GND), U12.7 (PAD)
- net +5VD: now reaches J1.A4_B9 (VBUS), J1.B4_A9 (VBUS__1)
- net +5VD: now also U12.4 (EN), U12.6 (IN)
- net EPR_SBU1C: now reaches U3.1 (C_SBU1)
- net EPR_SBU2C: now reaches U3.2 (C_SBU2)
- no-connect marks 19 -> 21
Other:
- moved on the sheet: C1, C10, C11, C12, C13, C14, C15, C16, C17, C18, C19, C2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

Commit message: dcdc
Parts:
- added J5: 5V_OUT, Connector_AMASS:AMASS_XT30U-F_1x02_P5.0mm_Vertical, symbol Connector:Conn_01x02_Socket
Connections:
- net +5VD: now also J5.2 (Pin_2)
- net GND: now also J5.1 (Pin_1)
Other:
- moved on the sheet: U12

Commit message: dcdc
Parts:
- added C66: 100n, Capacitor_SMD:C_0402_1005Metric, symbol Device:C
- added R3: 7.87M, Resistor_SMD:R_0402_1005Metric, symbol Device:R
- added R37, R38: 10k, Resistor_SMD:R_0402_1005Metric, symbol Device:R
- added R4: 1.07M, Resistor_SMD:R_0402_1005Metric, symbol Device:R
Connections:
- net +10V: now also R3.1
- net +3V3: now also C66.1, R37.1, R38.1; no longer U1.26 (RUN)
- net +5V: no longer C2.1
- net +5VD: now also C2.1
- net GND: now also C66.2, R4.2
- net TLV_GPIO: no longer U1.41 (GPIO27_ADC1)
- net TLV_RESET: now also R37.2
- net V_CSD: now also U1.41 (GPIO27_ADC1)
- net at U10.2 (FB): now also R3.2, R4.1
- net MCLK_unused: no longer names the net of U1.43 (GPIO29_ADC3)
- net MCLK_unused: no longer U4.1 (MCLK_(1))
- new net: R38.2, U1.26 (RUN)
- no-connect marks 21 -> 25
Other:
- note added: "-> TO AIC3254"
- note added: "-> TO HUB75"
- note added: "-> TO PD CONTROLLER"
- moved on the sheet: C22, C23, C64, C65, U10

Commit message: dcdc
Parts:
- added R42, R43: 22k, Resistor_SMD:R_0402_1005Metric, symbol Device:R
Connections:
- net +5VD: now also R42.2, R43.1
- net VBUS: now also J2.A4_B9 (VBUS), J2.B4_A9 (VBUS__1)
- net at J1.A5 (CC1): now also R43.2
- net at J1.B5 (CC2): now also R42.1
- net at U11.18 (EN): now also U11.20 (PVIN), U11.21 (PVIN), U11.22 (PVIN)

Commit message: work
Parts:
- removed U11: LM76005QRNPRQ1, LM76005:RNP0030A, symbol LM76005:LM76005QRNPRQ1
- added U11: LM70660RRXR, ul_LM70660RRXR:RRX0029B-MFG, symbol LM70660:LM70660RRXR
- added U13: MP23ABS1TR, RHLGA5_STM, symbol MP23:MP23ABS1TR
Connections:
- net +3V3: now also U13.5 (VDD)
- net GND: now also U13.2 (GND), U13.3 (GND), U13.4 (GND)
- net VI_SENSE: now reaches U1.43 (GPIO29_ADC3)
- net MIC_OUT: now reaches U4.15 (IN2_L)
- net MIC_OUT: now also U13.1 (OUT)
- no-connect marks 25 -> 17

Commit message: work
Parts:
- added C67: 47nF, Capacitor_SMD:C_0402_1005Metric, symbol Device:C
Connections:
- net at U11.20 (SW1): now also C67.1
- net at U11.4 (CBOOT): now also C67.2
Changed lines of the file:
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@@
 	(wire
 		(pts
+			(xy 195.58 45.72) (xy 198.12 45.72)
+		)
+		(stroke
+			(width 0)
+			(type default)
+		)
+	)
+	(wire
+		(pts
 			(xy 532.13 153.67) (xy 532.13 156.21)
 		)
@@
 	(wire
 		(pts
+			(xy 195.58 50.8) (xy 208.28 50.8)
+		)
+		(stroke
+			(width 0)
+			(type default)
+		)
+	)
+	(wire
+		(pts
 			(xy 260.35 433.07) (xy 275.59 433.07)
 		)
@@
 	(wire
 		(pts
+			(xy 208.28 45.72) (xy 205.74 45.72)
+		)
+		(stroke
+			(width 0)
+			(type default)
+		)
+	)
+	(wire
+		(pts
 			(xy 229.87 379.73) (xy 229.87 367.03)
 		)
@@
 	(wire
 		(pts
+			(xy 208.28 50.8) (xy 208.28 45.72)
+		)
+		(stroke
+			(width 0)
+			(type default)
+		)
+	)
+	(wire
+		(pts
 			(xy 386.08 48.26) (xy 392.43 48.26)
 		)
@@
 					(unit 1)
 				)
+			)
+		)
+	)
+	(symbol
+		(lib_id "Device:C")
+		(at 201.93 45.72 270)
+		(unit 1)
+		(exclude_from_sim no)
+		(in_bom yes)
+		(on_board yes)
+		(dnp no)
+		(property "Reference" "C67"
+			(at 202.946 47.244 90)
+			(effects
+				(font
+					(size 1.27 1.27)
+				)
+				(justify left)
+			)
+		)
+		(property "Value" "47nF"
+			(at 197.104 47.244 90)
+			(effects
+				(font
+					(size 1.27 1.27)
+				)
+				(justify left)
+			)
+		)
+		(property "Footprint" "Capacitor_SMD:C_0402_1005Metric"
+			(at 198.12 46.6852 0)
+			(effects
+				(font
+					(size 1.27 1.27)
+				)
+				(hide yes)
+			)
+		)
+		(property "Datasheet" "~"
+			(at 201.93 45.72 0)
+			(effects
+				(font
+					(size 1.27 1.27)
+				)
+				(hide yes)
+			)
+		)
+		(property "Description" "Unpolarized capacitor"
+			(at 201.93 45.72 0)
+			(effects
+				(font
+					(size 1.27 1.27)
+				)
+				(hide yes)
+			)
+		)
+		(pin "2"
+		)
+		(pin "1"
+		)
+		(instances
+			(project "ioAmp200W"
+				(path "/4f3b51aa-8e6e-4521-ad6c-a7e6e194e2a4"
+					(reference "C67")
+					(unit 1)
+				)
