File: board/ioAmp200W.kicad_sch (KiCad schematic)
At the start: 152 parts, among them J1 USB4105-GF-A-120, J2 USB4105-GF-A-120, J3 Speaker_Out, J4 SM03B-SRSS-TB, J5 5V_OUT, SW1 SW_Push, U1 RP2350_60QFN, U10 TPS7A1601DRBR, U11 LM70660RRXR, U12 TLV75733PDRVR, U14 MA5332MS, U15 TAD5112, U2 TPS26750SRSMR, U3 TPD4S480RUKR, U4 LP5912-3.3DRV, U5 MA5332MS, U6 SN74AHCT245RGYR, U7 SN74AHCT245RGYR, U8 Winbond W25Q32JVUUIQ, U9 TLV9162IDSGR, Y1 ABM8-272-T3

Commit message: work
Parts:
- removed R38: 10k, Resistor_SMD:R_0402_1005Metric, symbol Device:R
- added C74, C76, C78: 0.1u, Capacitor_SMD:C_0402_1005Metric, symbol Device:C
- added C75, C77: 10u, Capacitor_SMD:C_0402_1005Metric, symbol Device:C
- U10: footprint TPS26750SRSMR:VQFN32_RSM_TEX -> TPS7A:DRB0008B
Connections:
- net +3V3: now also U1.26 (RUN), C76.1, C77.1
- net +5VD: now also C74.1, C75.1, C78.1
- net AMP_CLIP: no longer U1.40 (GPIO26_ADC0)
- net GND: now also C74.2, C75.2, C76.2, C77.2, C78.2
- net I2S_Bclk: now also U1.5 (GPIO3); no longer U1.2 (GPIO0)
- net I2S_Din: now also U1.2 (GPIO0); no longer U1.5 (GPIO3)
- net I2S_Dout: now also U1.3 (GPIO1); no longer U1.4 (GPIO2)
- net I2S_Fsync: now also U1.4 (GPIO2); no longer U1.3 (GPIO1)
- net TAD_GPIO2: now reaches U1.10 (GPIO7)
- net TAD_GPIO2: now also U15.10 (GPIO2)
- net TPS_GPIO1: now reaches U1.12 (GPIO8)
- net TPS_GPIO2: now reaches U1.13 (GPIO9)
- net TPS_I2C_SDA: now reaches U1.14 (GPIO10)
- net TPS_I2C_SCL: now reaches U1.15 (GPIO11)
- net SPKR_SENSE-: now reaches U1.43 (GPIO29_ADC3)
- net TAD_GPIO1: now reaches U1.9 (GPIO6)
- net TAD_GPIO1: now also U15.9 (GPIO1)
- net CLIP: now reaches U14.1 (CLIP)
- net CLIP: now also U1.40 (GPIO26_ADC0)
- net I2C_SCL renamed TAD_I2C_SCL
- net I2C_SDA renamed TAD_I2C_SDA
- net VI_SENSE renamed SPKR_SENSE+
- no-connect marks 23 -> 21
Other:
- moved on the sheet: C42, C43, C57, C58, C59, C60, C61, C62, C63, D1, R23, R24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

Commit message: work
Parts:
- added C79, C80, C81, C82: 1u, Capacitor_SMD:C_0402_1005Metric, symbol Device:C
Connections:
- net +3V3: now also C80.1
- net +5VD: now also C79.1, C81.1
- net GND: now also C79.2, C80.2, C81.2, C82.2
- net LN_3V3: now also C82.1
Other:
- moved on the sheet: C64, C65, C66, C74, C75, C77, C78

Commit message: buck
Parts:
- added C83, C84, C85, C86, C88, C89, C90, C91: 47u, Capacitor_SMD:C_0402_1005Metric, symbol Device:C
- added C87: 4.7u, Capacitor_SMD:C_0402_1005Metric, symbol Device:C
- added C92, C95: 0.1u, Capacitor_SMD:C_0402_1005Metric, symbol Device:C
- added C93: 6.8n, Capacitor_SMD:C_0402_1005Metric, symbol Device:C
- added C94: 4.7p, Capacitor_SMD:C_0402_1005Metric, symbol Device:C
- added L4: 3.3u, Capacitor_SMD:C_0402_1005Metric, symbol Device:L
- added R47: 1, Resistor_SMD:R_0402_1005Metric, symbol Device:R
- added R48: 5m, Resistor_SMD:R_0402_1005Metric, symbol Device:R
- added R49, R51: 100k, Resistor_SMD:R_0402_1005Metric, symbol Device:R
- added R50: 20.5k, Resistor_SMD:R_0402_1005Metric, symbol Device:R
- added R52: 19.1k, Resistor_SMD:R_0402_1005Metric, symbol Device:R
- added R53: 5.76k, Resistor_SMD:R_0402_1005Metric, symbol Device:R
- added R54: 29.4k, Resistor_SMD:R_0402_1005Metric, symbol Device:R
- added R55: 54.9k, Resistor_SMD:R_0402_1005Metric, symbol Device:R
Connections:
- net +5VD: now also U11.12 (VOUT), C83.1, C84.1, C85.1, C86.1, R48.1, R51.1
- net GND: now also U11.17 (AGND), U11.23 (PGND1), U11.24 (PGND2), U11.25 (PGND3), U11.26 (PGND4), U11.30 (PGND), U11.6 (BIAS), U11.8 (PFM_SYNCIN), C83.2, C84.2, C85.2, C86.2, C87.2, C88.2, C89.2, C90.2, C91.2, C92.2, C93.2, C94.2, C95.2, R50.2, R52.2, R54.1, R55.1
- net VBUS: now also U11.1 (VIN4), U11.2 (VIN5), U11.27 (VIN1), U11.28 (VIN2), U11.29 (VIN3), U11.3 (VIN6), C88.1, C89.1, C90.1, C91.1, C92.1, R49.2
- net at C67.1: now also R47.1; no longer U11.20 (SW1)
- net at U11.11 (ISNS+): now also L4.2, R48.2
- net at U11.13 (CONFIG): now also R54.2
- net at U11.14 (RT): now also R55.2
- net at U11.15 (EXTCOMP): now also C94.1, R53.2
- net at U11.16 (FB): now also R51.2, R52.1
- net at U11.18 (VDDA): now also C95.1
- net at U11.19 (VCC): now also C87.1
- net at U11.21 (SW2): now also U11.20 (SW1), U11.22 (SW3), U11.5 (SW4), L4.1, R47.2
- net at U11.9 (EN_UVLO): now also R49.1, R50.1
- new net: C93.1, R53.1
- no-connect marks 21 -> 23
Other:
- moved on the sheet: C74, C75, C76, C77, C79, C80, U12

Commit message: verifybuck
Parts:
- C88, C89, C90, C91: value 47u -> 4.7u
- C94: value 4.7p -> 47p
Other:
- moved on the sheet: C74, C75, C76, C77, C79, C80, J5, U12

Commit message: verifybuck
Parts:
- U14: footprint (none) -> MA5332MS_footprint:IFX-PG-IQFN-42-1-V
- U5: footprint MA5332MS_footprint:IFX-PG-IQFN-42-1-V -> a
Changed lines of the file:
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@@
 	)
 	(junction
-		(at 459.74 668.02)
-		(diameter 0)
-		(color 0 0 0 0)
-	)
-	(junction
 		(at 233.68 66.04)
 		(diameter 0)
@@
 	(wire
 		(pts
-			(xy 459.74 668.02) (xy 459.74 681.99)
-		)
-		(stroke
-			(width 0)
-			(type default)
-		)
-	)
-	(wire
-		(pts
 			(xy 205.74 346.71) (xy 205.74 367.03)
 		)
@@
 	(wire
 		(pts
-			(xy 461.01 668.02) (xy 459.74 668.02)
-		)
-		(stroke
-			(width 0)
-			(type default)
-		)
-	)
-	(wire
-		(pts
 			(xy 386.08 48.26) (xy 392.43 48.26)
 		)
@@
 	(wire
 		(pts
-			(xy 459.74 655.32) (xy 459.74 668.02)
-		)
-		(stroke
-			(width 0)
-			(type default)
-		)
-	)
-	(wire
-		(pts
 			(xy 560.07 43.18) (xy 579.12 43.18)
 		)
@@
 			)
 		)
-		(property "Footprint" "MA5332MS_footprint:IFX-PG-IQFN-42-1-V"
+		(property "Footprint" "a"
 			(at 532.13 330.2 0)
 			(hide yes)
@@
 	)
 	(symbol
+		(lib_id "power:GND")
+		(at 459.74 681.99 270)
+		(unit 1)
+		(body_style 1)
+		(exclude_from_sim no)
+		(in_bom yes)
+		(on_board yes)
+		(in_pos_files yes)
+		(dnp no)
+		(fields_autoplaced yes)
+		(property "Reference" "#PWR0119"
+			(at 453.39 681.99 0)
+			(hide yes)
+			(show_name no)
+			(do_not_autoplace no)
+			(effects
+				(font
+					(size 1.27 1.27)
+				)
+			)
+		)
+		(property "Value" "GND"
+			(at 455.93 681.9899 90)
+			(show_name no)
+			(do_not_autoplace no)
+			(effects
+				(font
+					(size 1.27 1.27)
+				)
+				(justify right)
+			)
+		)
+		(property "Footprint" ""
+			(at 459.74 681.99 0)
+			(hide yes)
+			(show_name no)
+			(do_not_autoplace no)
+			(effects
+				(font
+					(size 1.27 1.27)
+				)
+			)
+		)
+		(property "Datasheet" ""
+			(at 459.74 681.99 0)
+			(hide yes)
+			(show_name no)
+			(do_not_autoplace no)
+			(effects
+				(font
+					(size 1.27 1.27)
+				)
+			)
+		)
+		(property "Description" "Power symbol creates a global label with name \"GND\" , ground"
+			(at 459.74 681.99 0)
+			(hide yes)
+			(show_name no)
+			(do_not_autoplace no)
+			(effects
+				(font
+					(size 1.27 1.27)
+				)
+			)
+		)
+		(pin "1"
+		)
+		(instances
+			(project "ioAmp200W"
+				(path "/4f3b51aa-8e6e-4521-ad6c-a7e6e194e2a4"
+					(reference "#PWR0119")
+					(unit 1)
+				)
+			)
+		)
+	)
+	(symbol
 		(lib_id "Diode:1N4148")
 		(at 549.91 322.58 0)
@@
 	)
 	(symbol
+		(lib_id "power:GND")
+		(at 459.74 655.32 270)
+		(unit 1)
+		(body_style 1)
+		(exclude_from_sim no)
+		(in_bom yes)
+		(on_board yes)
+		(in_pos_files yes)
+		(dnp no)
+		(fields_autoplaced yes)
+		(property "Reference" "#PWR071"
+			(at 453.39 655.32 0)
+			(hide yes)
+			(show_name no)
+			(do_not_autoplace no)
+			(effects
+				(font
+					(size 1.27 1.27)
+				)
+			)
+		)
+		(property "Value" "GND"
+			(at 455.93 655.3199 90)
+			(show_name no)
+			(do_not_autoplace no)
+			(effects
+				(font
+					(size 1.27 1.27)
+				)
+				(justify right)
+			)
+		)
+		(property "Footprint" ""
+			(at 459.74 655.32 0)
+			(hide yes)
+			(show_name no)
+			(do_not_autoplace no)
+			(effects
+				(font
+					(size 1.27 1.27)
+				)
+			)
+		)
+		(property "Datasheet" ""
+			(at 459.74 655.32 0)
+			(hide yes)
+			(show_name no)
+			(do_not_autoplace no)
+			(effects
+				(font
+					(size 1.27 1.27)
+				)
+			)
+		)
+		(property "Description" "Power symbol creates a global label with name \"GND\" , ground"
+			(at 459.74 655.32 0)
+			(hide yes)
+			(show_name no)
+			(do_not_autoplace no)
+			(effects
+				(font
+					(size 1.27 1.27)
+				)
+			)
+		)
+		(pin "1"
+		)
+		(instances
+			(project "ioAmp200W"
+				(path "/4f3b51aa-8e6e-4521-ad6c-a7e6e194e2a4"
+					(reference "#PWR071")
+					(unit 1)
+				)
+			)
+		)
+	)
+	(symbol
 		(lib_id "Device:C")
 		(at 114.3 46.99 0)
@@
 			)
 		)
-		(property "Footprint" ""
+		(property "Footprint" "MA5332MS_footprint:IFX-PG-IQFN-42-1-V"
 			(at 499.11 635 0)
 			(hide yes)
@@
 					(unit 1)
 				)
-			)
-		)
-	)
-	(symbol
-		(lib_id "power:GND")
-		(at 461.01 668.02 90)
-		(unit 1)
-		(body_style 1)
-		(exclude_from_sim no)
-		(in_bom yes)
-		(on_board yes)
-		(in_pos_files yes)
-		(dnp no)
-		(fields_autoplaced yes)
-		(property "Reference" "#PWR071"
-			(at 467.36 668.02 0)
-			(hide yes)
-			(show_name no)
-			(do_not_autoplace no)
-			(effects
-				(font
-					(size 1.27 1.27)
-				)
-			)
-		)
-		(property "Value" "GND"
-			(at 464.82 668.0199 90)
-			(show_name no)
-			(do_not_autoplace no)
-			(effects
-				(font
-					(size 1.27 1.27)
-				)
-				(justify right)
-			)
-		)
-		(property "Footprint" ""
-			(at 461.01 668.02 0)
-			(hide yes)
-			(show_name no)
-			(do_not_autoplace no)
-			(effects
-				(font
-					(size 1.27 1.27)
-				)
-			)
-		)
-		(property "Datasheet" ""
-			(at 461.01 668.02 0)
-			(hide yes)
-			(show_name no)
-			(do_not_autoplace no)
-			(effects
-				(font
-					(size 1.27 1.27)
-				)
-			)
-		)
-		(property "Description" "Power symbol creates a global label with name \"GND\" , ground"
-			(at 461.01 668.02 0)
-			(hide yes)
-			(show_name no)
-			(do_not_autoplace no)
-			(effects
-				(font
-					(size 1.27 1.27)
-				)
-			)
-		)
-		(pin "1"
-		)
-		(instances
-			(project "ioAmp200W"
-				(path "/4f3b51aa-8e6e-4521-ad6c-a7e6e194e2a4"
-					(reference "#PWR071")
-					(unit 1)
-				)

Commit message: verifybuck
Parts:
- C83, C84, C85, C86: footprint Capacitor_SMD:C_0402_1005Metric -> Capacitor_SMD:C_1210_3225Metric; LCSC (none) -> C440151
- C87, C88, C89, C90: footprint Capacitor_SMD:C_0402_1005Metric -> Capacitor_SMD:C_1210_3225Metric; LCSC (none) -> C913445
- C91: footprint Capacitor_SMD:C_0402_1005Metric -> Capacitor_SMD:C_1210_3225Metric
- L4: footprint Capacitor_SMD:C_0402_1005Metric -> Inductor_SMD:L_Bourns_SRP7028A_7.3x6.6mm; LCSC (none) -> C3040366
- R48: footprint Resistor_SMD:R_0402_1005Metric -> Resistor_SMD:R_1206_3216Metric; LCSC (none) -> C6973817
- SW1: LCSC (none) -> C720477
Changed lines of the file:
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@@
 			)
 		)
-		(property "Footprint" "Capacitor_SMD:C_0402_1005Metric"
+		(property "Footprint" "Capacitor_SMD:C_1210_3225Metric"
 			(at 247.3452 74.93 0)
 			(hide yes)
@@
 			)
 		)
+		(property "LCSC" "C440151"
+			(at 246.38 71.12 90)
+			(hide yes)
+			(show_name no)
+			(do_not_autoplace no)
+			(effects
+				(font
+					(size 1.27 1.27)
+				)
+			)
+		)
 		(pin "2"
 		)
@@
 			)
 		)
-		(property "Footprint" "Resistor_SMD:R_0402_1005Metric"
+		(property "Footprint" "Resistor_SMD:R_1206_3216Metric"
 			(at 219.71 64.262 90)
 			(hide yes)
@@
 			)
 		)
+		(property "LCSC" "C6973817"
+			(at 219.71 66.04 90)
+			(hide yes)
+			(show_name no)
+			(do_not_autoplace no)
+			(effects
+				(font
+					(size 1.27 1.27)
+				)
+			)
+		)
 		(pin "2"
 		)
@@
 			)
 		)
-		(property "Footprint" "Capacitor_SMD:C_0402_1005Metric"
+		(property "Footprint" "Capacitor_SMD:C_1210_3225Metric"
 			(at 234.6452 74.93 0)
 			(hide yes)
@@
 			)
 		)
+		(property "LCSC" "C440151"
+			(at 233.68 71.12 90)
+			(hide yes)
+			(show_name no)
+			(do_not_autoplace no)
+			(effects
+				(font
+					(size 1.27 1.27)
+				)
+			)
+		)
 		(pin "2"
 		)
@@
 			)
 		)
-		(property "Footprint" "Capacitor_SMD:C_0402_1005Metric"
+		(property "Footprint" "Capacitor_SMD:C_1210_3225Metric"
 			(at 121.6152 50.8 0)
 			(hide yes)
@@
 			)
 		)
+		(property "LCSC" "C913445"
+			(at 120.65 46.99 90)
+			(hide yes)
+			(show_name no)
+			(do_not_autoplace no)
+			(effects
+				(font
+					(size 1.27 1.27)
+				)
+			)
+		)
 		(pin "2"
 		)
@@
 		)
 		(property "Value" "6.8n"
-			(at 124.714 85.344 90)
+			(at 124.968 85.344 90)
 			(show_name no)
 			(do_not_autoplace no)
@@
 			)
 		)
-		(property "Footprint" "Capacitor_SMD:C_0402_1005Metric"
+		(property "Footprint" "Capacitor_SMD:C_1210_3225Metric"
 			(at 115.2652 50.8 0)
 			(hide yes)
@@
 			)
 		)
+		(property "LCSC" "C913445"
+			(at 114.3 46.99 90)
+			(hide yes)
+			(show_name no)
+			(do_not_autoplace no)
+			(effects
+				(font
+					(size 1.27 1.27)
+				)
+			)
+		)
 		(pin "2"
 		)
@@
 			)
 		)
-		(property "Footprint" "Capacitor_SMD:C_0402_1005Metric"
+		(property "Footprint" "Inductor_SMD:L_Bourns_SRP7028A_7.3x6.6mm"
 			(at 207.01 66.04 0)
 			(hide yes)
@@
 			)
 		)
+		(property "LCSC" "C3040366"
+			(at 207.01 66.04 90)
+			(hide yes)
+			(show_name no)
+			(do_not_autoplace no)
+			(effects
+				(font
+					(size 1.27 1.27)
+				)
+			)
+		)
 		(pin "1"
 		)
@@
 			)
 		)
-		(property "Footprint" "Capacitor_SMD:C_0402_1005Metric"
+		(property "Footprint" "Capacitor_SMD:C_1210_3225Metric"
 			(at 108.9152 50.8 0)
 			(hide yes)
@@
 			)
 		)
+		(property "LCSC" "C913445"
+			(at 107.95 46.99 90)
+			(hide yes)
+			(show_name no)
+			(do_not_autoplace no)
+			(effects
+				(font
+					(size 1.27 1.27)
+				)
+			)
+		)
 		(pin "2"
 		)
@@
 			)
 		)
-		(property "Footprint" "Capacitor_SMD:C_0402_1005Metric"
+		(property "Footprint" "Capacitor_SMD:C_1210_3225Metric"
 			(at 228.2952 74.93 0)
 			(hide yes)
@@
 			)
 		)
+		(property "LCSC" "C440151"
+			(at 227.33 71.12 90)
+			(hide yes)
+			(show_name no)
+			(do_not_autoplace no)
+			(effects
+				(font
+					(size 1.27 1.27)
+				)
+			)
+		)
 		(pin "2"
 		)
@@
 			)
 		)
+		(property "LCSC" "C720477"
+			(at 158.115 416.56 90)
+			(hide yes)
+			(show_name no)
+			(do_not_autoplace no)
+			(effects
+				(font
+					(size 1.27 1.27)
+				)
+			)
+		)
 		(pin "1"
 		)
@@
 			)
 		)
-		(property "Footprint" "Capacitor_SMD:C_0402_1005Metric"
+		(property "Footprint" "Capacitor_SMD:C_1210_3225Metric"
 			(at 127.9652 50.8 0)
 			(hide yes)
@@
 			)
 		)
-		(property "Footprint" "Capacitor_SMD:C_0402_1005Metric"
+		(property "Footprint" "Capacitor_SMD:C_1210_3225Metric"
 			(at 137.16 63.1952 0)
 			(hide yes)
@@
 			)
 		)
+		(property "LCSC" "C913445"
+			(at 140.97 62.23 90)
+			(hide yes)
+			(show_name no)
+			(do_not_autoplace no)
+			(effects
+				(font
+					(size 1.27 1.27)
+				)
+			)
+		)
 		(pin "2"
 		)
@@
 			)
 		)
-		(property "Footprint" "Capacitor_SMD:C_0402_1005Metric"
+		(property "Footprint" "Capacitor_SMD:C_1210_3225Metric"
 			(at 240.9952 74.93 0)
 			(hide yes)
@@
 			(hide yes)
 			(show_name no)
+			(do_not_autoplace no)
+			(effects
+				(font
+					(size 1.27 1.27)
+				)
+			)
+		)
+		(property "LCSC" "C440151"
+			(at 240.03 71.12 90)
+			(hide yes)
+			(show_name no)

Commit message: update
Connections:
- net TPS_GPIO2 is gone; now on net TPS_I2C_IRQ: U1.13 (GPIO9)
- net EPR_DN: now also U2.23 (GPIO5/USB_N/LD2)
- net EPR_DP: now also U2.22 (GPIO4/USB_P/LD1)
- net TPS_I2C_SCL: now also U2.9 (I2CT_SCL)
- net TPS_I2C_SDA: now also U2.8 (I2CT_SDA)
- net TPS_I2C_IRQ: now reaches U2.10 (*I2CT_IRQ)
- net at U2.26 (VBUS): now also U2.27 (VBUS)
- net at U2.28 (PP5V): now also U2.29 (PP5V)
- no-connect marks 23 -> 25
Changed lines of the file:
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@@
 	)
 	(junction
+		(at 234.95 228.6)
+		(diameter 0)
+		(color 0 0 0 0)
+	)
+	(junction
 		(at 525.78 332.74)
 		(diameter 0)
@@
 	)
 	(junction
+		(at 234.95 223.52)
+		(diameter 0)
+		(color 0 0 0 0)
+	)
+	(junction
 		(at 608.33 369.57)
 		(diameter 0)
@@
 	)
 	(no_connect
+		(at 184.15 233.68)
+	)
+	(no_connect
 		(at 645.16 774.7)
 	)
@@
 	)
 	(no_connect
+		(at 184.15 226.06)
+	)
+	(no_connect
 		(at 461.01 199.39)
 	)
@@
 	(wire
 		(pts
+			(xy 227.33 252.73) (xy 234.95 252.73)
+		)
+		(stroke
+			(width 0)
+			(type default)
+		)
+	)
+	(wire
+		(pts
 			(xy 77.47 67.31) (xy 85.09 67.31)
 		)
@@
 	(wire
 		(pts
+			(xy 323.85 232.41) (xy 311.15 232.41)
+		)
+		(stroke
+			(width 0)
+			(type default)
+		)
+	)
+	(wire
+		(pts
 			(xy 378.46 664.21) (xy 397.51 664.21)
 		)
@@
 	(wire
 		(pts
+			(xy 234.95 223.52) (xy 234.95 224.79)
+		)
+		(stroke
+			(width 0)
+			(type default)
+		)
+	)
+	(wire
+		(pts
 			(xy 260.35 407.67) (xy 275.59 407.67)
 		)
@@
 	(wire
 		(pts
+			(xy 234.95 247.65) (xy 218.44 247.65)
+		)
+		(stroke
+			(width 0)
+			(type default)
+		)
+	)
+	(wire
+		(pts
 			(xy 527.05 347.98) (xy 511.81 347.98)
 		)
@@
 	(wire
 		(pts
+			(xy 322.58 250.19) (xy 311.15 250.19)
+		)
+		(stroke
+			(width 0)
+			(type default)
+		)
+	)
+	(wire
+		(pts
 			(xy 527.05 756.92) (xy 527.05 755.65)
 		)
@@
 	(wire
 		(pts
+			(xy 224.79 240.03) (xy 234.95 240.03)
+		)
+		(stroke
+			(width 0)
+			(type default)
+		)
+	)
+	(wire
+		(pts
 			(xy 525.78 331.47) (xy 525.78 332.74)
 		)
@@
 	(wire
 		(pts
+			(xy 323.85 229.87) (xy 311.15 229.87)
+		)
+		(stroke
+			(width 0)
+			(type default)
+		)
+	)
+	(wire
+		(pts
 			(xy 260.35 448.31) (xy 275.59 448.31)
 		)
@@
 	(wire
 		(pts
+			(xy 224.79 237.49) (xy 234.95 237.49)
+		)
+		(stroke
+			(width 0)
+			(type default)
+		)
+	)
+	(wire
+		(pts
 			(xy 554.99 355.6) (xy 554.99 379.73)
 		)
@@
 	(wire
 		(pts
+			(xy 335.28 245.11) (xy 335.28 252.73)
+		)
+		(stroke
+			(width 0)
+			(type default)
+		)
+	)
+	(wire
+		(pts
 			(xy 173.99 356.87) (xy 173.99 359.41)
 		)
@@
 	(wire
 		(pts
+			(xy 223.52 223.52) (xy 234.95 223.52)
+		)
+		(stroke
+			(width 0)
+			(type default)
+		)
+	)
+	(wire
+		(pts
 			(xy 457.2 687.07) (xy 457.2 690.88)
 		)
@@
 	(wire
 		(pts
+			(xy 218.44 247.65) (xy 218.44 252.73)
+		)
+		(stroke
+			(width 0)
+			(type default)
+		)
+	)
+	(wire
+		(pts
 			(xy 260.35 400.05) (xy 275.59 400.05)
 		)
@@
 	(wire
 		(pts
+			(xy 220.98 228.6) (xy 234.95 228.6)
+		)
+		(stroke
+			(width 0)
+			(type default)
+		)
+	)
+	(wire
+		(pts
 			(xy 149.86 389.89) (xy 149.86 388.62)
 		)
@@
 	(wire
 		(pts
+			(xy 323.85 234.95) (xy 311.15 234.95)
+		)
+		(stroke
+			(width 0)
+			(type default)
+		)
+	)
+	(wire
+		(pts
 			(xy 158.115 421.64) (xy 158.115 424.18)
 		)
@@
 	(wire
 		(pts
+			(xy 234.95 212.09) (xy 215.9 212.09)
+		)
+		(stroke
+			(width 0)
+			(type default)
+		)
+	)
+	(wire
+		(pts
 			(xy 553.72 762) (xy 551.18 762)
 		)
@@
 	(wire
 		(pts
+			(xy 234.95 227.33) (xy 234.95 228.6)
+		)
+		(stroke
+			(width 0)
+			(type default)
+		)
+	)
+	(wire
+		(pts
 			(xy 184.15 375.92) (xy 184.15 377.19)
 		)
@@
 	(wire
 		(pts
+			(xy 215.9 212.09) (xy 215.9 214.63)
+		)
+		(stroke
+			(width 0)
+			(type default)
+		)
+	)
+	(wire
+		(pts
 			(xy 567.69 353.06) (xy 567.69 364.49)
 		)
@@
 	(wire
 		(pts
+			(xy 322.58 247.65) (xy 311.15 247.65)
+		)
+		(stroke
+			(width 0)
+			(type default)
+		)
+	)
+	(wire
+		(pts
 			(xy 205.74 367.03) (xy 205.74 379.73)
 		)
@@
 	(wire
 		(pts
+			(xy 234.95 228.6) (xy 234.95 229.87)
+		)
+		(stroke
+			(width 0)
+			(type default)
+		)
+	)
+	(wire
+		(pts
 			(xy 575.31 373.38) (xy 576.58 373.38)
 		)
@@
 	(wire
 		(pts
+			(xy 234.95 222.25) (xy 234.95 223.52)
+		)
+		(stroke
+			(width 0)
+			(type default)
+		)
+	)
+	(wire
+		(pts
 			(xy 165.1 388.62) (xy 165.1 389.89)
 		)
@@
 	(wire
 		(pts
+			(xy 311.15 245.11) (xy 335.28 245.11)
+		)
+		(stroke
+			(width 0)
+			(type default)
+		)
+	)
+	(wire
+		(pts
 			(xy 295.91 675.64) (xy 302.26 675.64)
 		)
@@
 		)
 	)
+	(label "TPS_I2C_SCL"
+		(at 323.85 232.41 180)
+		(effects
+			(font
+				(size 1.27 1.27)
+			)
+			(justify right bottom)
+		)
+	)
+	(label "EPR_DP"
+		(at 224.79 240.03 0)
+		(effects
+			(font
+				(size 1.27 1.27)
+			)
+			(justify left bottom)
+		)
+	)
 	(label "ROW_A"
 		(at 275.59 445.77 180)
@@
 		)
 	)
-	(label "TPS_I2C_SCL"
-		(at 279.4 193.04 180)
-		(effects
-			(font
-				(size 1.27 1.27)
-			)
-			(justify right bottom)
-		)
-	)
 	(label "B0"
 		(at 275.59 433.07 180)
@@
 		)
 	)
-	(label "STB"
-		(at 275.59 458.47 180)
+	(label "EPR_DN"
+		(at 224.79 237.49 0)
 		(effects
 			(font
 				(size 1.27 1.27)
 			)
-			(justify right bottom)
+			(justify left bottom)
 		)
 	)
-	(label "TPS_GPIO2"
-		(at 285.75 420.37 180)
+	(label "STB"
+		(at 275.59 458.47 180)
 		(effects
 			(font
@@
 		)
 	)
-	(label "TPS_I2C_SDA"
-		(at 279.4 190.5 180)
-		(effects
-			(font
-				(size 1.27 1.27)
-			)
-			(justify right bottom)
-		)
-	)
 	(label "ROW_A_5V"
 		(at 462.28 96.52 0)
@@
 		)
 	)
+	(label "TPS_I2C_IRQ"
+		(at 285.75 420.37 180)
+		(effects
+			(font
+				(size 1.27 1.27)
+			)
+			(justify right bottom)
+		)
+	)
 	(label "VREG_AVDD"
 		(at 184.785 375.92 0)
@@
 		)
 	)
-	(label "TPS_GPIO2"
-		(at 279.4 187.96 180)
-		(effects
-			(font
-				(size 1.27 1.27)
-			)
-			(justify right bottom)
-		)
-	)
 	(label "ROW_E_5V"
 		(at 382.27 55.88 0)
@@
 		)
 	)
+	(label "TPS_I2C_IRQ"
+		(at 323.85 234.95 180)
+		(effects
+			(font
+				(size 1.27 1.27)
+			)
+			(justify right bottom)
+		)
+	)
 	(label "ROW_D"
 		(at 571.5 53.34 180)
@@
 		(effects
 			(font
+				(size 1.27 1.27)
+			)
+			(justify right bottom)
+		)
+	)
+	(label "TPS_I2C_SDA"
+		(at 323.85 229.87 180)
+		(effects
+			(font

Commit message: summer_start
Parts:
- removed C64, C65, C75, C77: 10u, Capacitor_SMD:C_0402_1005Metric, symbol Device:C
- removed C66, C74, C76, C78: 0.1u, Capacitor_SMD:C_0402_1005Metric, symbol Device:C
- removed C79, C80, C81, C82: 1u, Capacitor_SMD:C_0402_1005Metric, symbol Device:C
- added C100, C101, C102, C103, C96, C97, C98, C99: 4.7u, Capacitor_SMD:C_1210_3225Metric, symbol Device:C
Connections:
- net +3V3: now also C98.1, C99.1
- net +5VD: now also C102.1, C103.1, C96.1, C97.1
- net GND: now also U15.11 (GPO1), U15.12 (GPI1), C100.2, C101.2, C102.2, C103.2, C96.2, C97.2, C98.2, C99.2
- net LN_3V3: now also C100.1, C101.1
- no-connect marks 25 -> 23
Other:
- moved on the sheet: J5, U12, U4
